Commit message: Fix warnings: joint limits, JSB interfaces, controller_manager name, base_footprint

File: lepantilt_description/urdf/pantilt.common.xacro (robot description, xacro)
@@ -9,5 +9,5 @@
   <xacro:property name="pan_offset_rx" value="${pi/2}"/>
   <xacro:property name="pan_offset_rz" value="${pi/2}"/>
-  <!-- Pan joint origin (in reoriented pantilt_base_link frame) -->
+  <!-- Pan joint origin (in reoriented base_link frame) -->
   <xacro:property name="pan_joint_x" value="0.0452"/>
   <xacro:property name="pan_joint_z" value="0.0165"/>

File: lepantilt_description/urdf/pantilt.control.xacro (robot description, xacro)
@@ -19,4 +19,4 @@
   <xacro:property name="pan_joint_upper" value="2"/>
   <xacro:property name="tilt_joint_lower" value="${-pi/2}"/>
-  <xacro:property name="tilt_joint_upper" value="2"/>
+  <xacro:property name="tilt_joint_upper" value="${pi/2}"/>
 </robot>

File: lepantilt_description/urdf/pantilt.urdf (robot description, URDF)
Before this commit: robot lepantilt, 3 links, 2 joints
Links:
- removed link pantilt_base_link
- added link base_footprint
- added link base_link, mass 1.0; collision mesh filename=../meshes/pantilt_base.stl; visual mesh filename=../meshes/pan_motor.stl
Joints:
- added joint base_footprint_joint: type fixed, parent base_footprint, child base_link, origin xyz=0 0 0 rpy=0 0 0
- joint pan_joint: parent pantilt_base_link -> base_link

File: lepantilt_description/urdf/pantilt.urdf.xacro (robot description, xacro)
@@ -16,6 +16,8 @@
   </material>
   <!-- LINKS -->
-  <!-- Pantilt base link -->
-  <link name="pantilt_base_link">
+  <!-- Base footprint link (empty root — KDL does not support inertia on root link) -->
+  <link name="base_footprint"/>
+  <!-- Base link -->
+  <link name="base_link">
     <inertial>
       <mass value="1.0"/>
@@ -94,7 +96,13 @@
   </link>
   <!-- JOINTS -->
+  <!-- base_footprint fixed joint -->
+  <joint name="base_footprint_joint" type="fixed">
+    <parent link="base_footprint"/>
+    <child link="base_link"/>
+    <origin xyz="0 0 0" rpy="0 0 0"/>
+  </joint>
   <!-- Pan joint (revolute) -->
   <joint name="pan_joint" type="revolute">
-    <parent link="pantilt_base_link"/>
+    <parent link="base_link"/>
     <child link="pan_link"/>
     <origin xyz="${pan_joint_x} 0 ${pan_joint_z}" rpy="0 0 0"/>

Commit message: Add OAK-D camera support, switch tilt mesh to lite variant
- Add oak_d_s2.stl mesh for OAK-D S2 camera link
- Add tilt_joint_lite.stl (replaces tilt_joint_s2.stl) for lekiwi-lite variant
- Remove tilt_joint_s2.stl (no longer referenced)
- Update pantilt.common.xacro: add camera/tilt visual offsets for lite variant
- Update pantilt.urdf.xacro: add oak_d_s2 camera link, use tilt_joint_lite.stl
- Update pantilt.urdf: regenerated to match xacro changes
- Update pantilt.launch.py: clean up launch arguments
- Update package.xml: add depthai_descriptions dependency

File: lepantilt_description/urdf/pantilt.common.xacro (robot description, xacro)
@@ -24,3 +24,9 @@
   <xacro:property name="tilt_visual_y" value="${pan_joint_x + tilt_joint_x}"/>
   <xacro:property name="tilt_visual_z" value="-0.0002"/>
+  <!-- OAK-D-S2 camera mount offset (in tilt_link frame) -->
+  <xacro:property name="oak_pos_x" value="-0.03435"/>
+  <xacro:property name="oak_pos_y" value="-0.01"/>
+  <!-- OAK-D-S2 camera mount orientation (in tilt_link frame) -->
+  <xacro:property name="oak_roll" value="${-pi/2}"/>
+  <xacro:property name="oak_yaw"  value="${-pi/2}"/>
 </robot>

File: lepantilt_description/urdf/pantilt.urdf (robot description, URDF)
Before this commit: robot lepantilt, 4 links, 3 joints
Links:
- added link oak
- added link oak_imu_frame
- added link oak_left_camera_frame
- added link oak_left_camera_optical_frame
- added link oak_model_origin; visual mesh filename=../meshes/oak_d_s2.stl
- added link oak_rgb_camera_frame
- added link oak_rgb_camera_optical_frame
- added link oak_right_camera_frame
- added link oak_right_camera_optical_frame
- link tilt_link: geometry collision mesh filename=../meshes/tilt_joint_lite.stl; visual mesh filename=../meshes/tilt_joint_lite.stl
Joints:
- added joint oak_imu_joint: type fixed, parent oak, child oak_imu_frame, origin xyz=-0.008 -0.037945 -0.00079 rpy=3.1415926535897932 1.5707963267948966 0.0
- added joint oak_left_camera_joint: type fixed, parent oak, child oak_left_camera_frame, origin xyz=0 0.0375 0 rpy=0 0 0
- added joint oak_left_camera_optical_joint: type fixed, parent oak_left_camera_frame, child oak_left_camera_optical_frame, origin xyz=0 0 0 rpy=-1.5707963267948966 0.0 -1.5707963267948966
- added joint oak_model_origin_joint: type fixed, parent oak, child oak_model_origin, origin xyz=0 0 0 rpy=1.5707963267948966 0 1.5707963267948966
- added joint oak_mount_joint: type fixed, parent tilt_link, child oak, origin xyz=-0.03435 -0.01 0.0 rpy=-1.5707963267948966 0.0 -1.5707963267948966
- added joint oak_rgb_camera_joint: type fixed, parent oak, child oak_rgb_camera_frame, origin xyz=0 0 0 rpy=0 0 0
- added joint oak_rgb_camera_optical_joint: type fixed, parent oak_rgb_camera_frame, child oak_rgb_camera_optical_frame, origin xyz=0 0 0 rpy=-1.5707963267948966 0.0 -1.5707963267948966
- added joint oak_right_camera_joint: type fixed, parent oak, child oak_right_camera_frame, origin xyz=0 -0.0375 0 rpy=0 0 0
- added joint oak_right_camera_optical_joint: type fixed, parent oak_right_camera_frame, child oak_right_camera_optical_frame, origin xyz=0 0 0 rpy=-1.5707963267948966 0.0 -1.5707963267948966
- joint tilt_joint: limit lower=-1.5707963268 upper=2.0 effort=2.942 velocity=5.21553467881118 -> lower=-1.5707963268 upper=1.5707963268 effort=2.942 velocity=5.21553467881118

File: lepantilt_description/urdf/pantilt.urdf.xacro (robot description, xacro)
@@ -3,10 +3,9 @@
   <xacro:include filename="$(find lepantilt_description)/urdf/pantilt.common.xacro"/>
   <xacro:include filename="$(find lepantilt_description)/urdf/pantilt.control.xacro"/>
+  <xacro:include filename="$(find depthai_descriptions)/urdf/include/depthai_macro.urdf.xacro"/>
   <!-- Arguments (externally settable, default to property values in pantilt.control.xacro) -->
   <xacro:arg name="serial_port"    default="${serial_port}"/>
   <xacro:arg name="use_mock"       default="${use_mock}"/>
   <xacro:arg name="use_sync_write" default="${use_sync_write}"/>
-  <xacro:arg name="tilt"           default="s2"/>
-  <xacro:property name="tilt" value="tilt_joint_$(arg tilt)"/>
   <material name="light_grey">
     <color rgba="${light_grey_rgba}"/>
@@ -84,5 +83,5 @@
       <origin xyz="${tilt_visual_x} ${tilt_visual_y} ${tilt_visual_z}" rpy="${tilt_offset_rx} ${tilt_offset_ry} 0"/>
       <geometry>
-        <mesh filename="package://lepantilt_description/meshes/${tilt}.stl"/>
+        <mesh filename="package://lepantilt_description/meshes/tilt_joint_lite.stl"/>
       </geometry>
       <material name="light_grey"/>
@@ -91,5 +90,5 @@
       <origin xyz="${tilt_visual_x} ${tilt_visual_y} ${tilt_visual_z}" rpy="${tilt_offset_rx} ${tilt_offset_ry} 0"/>
       <geometry>
-        <mesh filename="package://lepantilt_description/meshes/${tilt}.stl"/>
+        <mesh filename="package://lepantilt_description/meshes/tilt_joint_lite.stl"/>
       </geometry>
     </collision>
@@ -117,4 +116,20 @@
     <axis xyz="0 0 1"/>
     <limit lower="${tilt_joint_lower}" upper="${tilt_joint_upper}" effort="${max_torque_nm}" velocity="${max_velocity_rads}"/>
+  </joint>
+  <!-- OAK-D-S2 camera (fixed to tilt_link via depthai_descriptions macro) -->
+  <xacro:depthai_camera
+    camera_name="oak"
+    camera_model="OAK-D-S2"
+    base_frame="oak"
+    parent="tilt_link"
+    cam_pos_x="${oak_pos_x}" cam_pos_y="${oak_pos_y}" cam_pos_z="0"
+    cam_roll="${oak_roll}" cam_pitch="0" cam_yaw="${oak_yaw}"
+    r="0.15" g="0.15" b="0.15" a="1.0"/>
+  <!-- OAK-D-S2 IMU frame (hardcoded until upstream depthai_descriptions adds OAK-D-S2 IMU support) -->
+  <link name="oak_imu_frame"/>
+  <joint name="oak_imu_joint" type="fixed">
+    <parent link="oak"/>
+    <child link="oak_imu_frame"/>
+    <origin xyz="-0.008 -0.037945 -0.00079" rpy="${pi} ${pi/2} 0"/>
   </joint>
   <!-- ROS 2 CONTROL -->
