Commit message: Replace oak_d_s2.stl with oakd_lite.stl (from depthai_descriptions)

File: lepantilt_description/urdf/pantilt.urdf (robot description, URDF)
Before this commit: robot lepantilt, 12 links, 11 joints
Links:
- link oak_model_origin: geometry visual mesh filename=../meshes/oakd_lite.stl

Commit message: Merge s2: use OAK-D-S2, tilt_joint.stl; remove lite variants

File: lepantilt_description/urdf/pantilt.urdf (robot description, URDF)
Before this commit: robot lepantilt, 12 links, 11 joints
Links:
- link oak_model_origin: geometry visual mesh filename=../meshes/oak_d_s2.stl
- link tilt_link: geometry collision mesh filename=../meshes/tilt_joint.stl; visual mesh filename=../meshes/tilt_joint.stl

File: lepantilt_description/urdf/pantilt.urdf.xacro (robot description, xacro)
@@ -83,5 +83,5 @@
       <origin xyz="${tilt_visual_x} ${tilt_visual_y} ${tilt_visual_z}" rpy="${tilt_offset_rx} ${tilt_offset_ry} 0"/>
       <geometry>
-        <mesh filename="package://lepantilt_description/meshes/tilt_joint_lite.stl"/>
+        <mesh filename="package://lepantilt_description/meshes/tilt_joint.stl"/>
       </geometry>
       <material name="light_grey"/>
@@ -90,5 +90,5 @@
       <origin xyz="${tilt_visual_x} ${tilt_visual_y} ${tilt_visual_z}" rpy="${tilt_offset_rx} ${tilt_offset_ry} 0"/>
       <geometry>
-        <mesh filename="package://lepantilt_description/meshes/tilt_joint_lite.stl"/>
+        <mesh filename="package://lepantilt_description/meshes/tilt_joint.stl"/>
       </geometry>
     </collision>
@@ -117,8 +117,8 @@
     <limit lower="${tilt_joint_lower}" upper="${tilt_joint_upper}" effort="${max_torque_nm}" velocity="${max_velocity_rads}"/>
   </joint>
-  <!-- OAK-D-LITE camera (fixed to tilt_link via depthai_descriptions macro) -->
+  <!-- OAK-D-S2 camera (fixed to tilt_link via depthai_descriptions macro) -->
   <xacro:depthai_camera
     camera_name="oak"
-    camera_model="OAK-D-LITE"
+    camera_model="OAK-D-S2"
     base_frame="oak"
     parent="tilt_link"
