Commit message: update urdf

File: lepantilt_description/urdf/pantilt.control.xacro (robot description, xacro)
@@ -1,9 +1,9 @@
 <?xml version="1.0"?>
 <robot xmlns:xacro="http://www.ros.org/wiki/xacro">
-  <!-- Shared hardware interface parameters (single STS servo bus) -->
-  <xacro:property name="serial_port" default="/dev/ttySERVO"/>
-  <xacro:property name="baud_rate" default="1000000"/>
-  <xacro:property name="use_mock" default="false"/>
-  <xacro:property name="use_sync_write" default="true"/>
+  <!-- Arguments (externally settable via command line) -->
+  <xacro:arg name="serial_port"    default="/dev/ttySERVO"/>
+  <xacro:arg name="baud_rate"      default="1000000"/>
+  <xacro:arg name="use_mock"       default="false"/>
+  <xacro:arg name="use_sync_write" default="true"/>
   <!-- Pantilt motor IDs and mode -->
   <xacro:property name="pan_motor_id" value="1"/>
@@ -20,3 +20,50 @@
   <xacro:property name="tilt_joint_lower" value="${-pi/2}"/>
   <xacro:property name="tilt_joint_upper" value="${pi/2}"/>
+  <!-- ROS 2 CONTROL -->
+  <ros2_control name="lepantilt_control" type="system">
+    <hardware>
+      <plugin>sts_hardware_interface/STSHardwareInterface</plugin>
+      <param name="serial_port">$(arg serial_port)</param>
+      <param name="baud_rate">$(arg baud_rate)</param>
+      <param name="communication_timeout_ms">100</param>
+      <param name="use_sync_write">$(arg use_sync_write)</param>
+      <param name="enable_mock_mode">$(arg use_mock)</param>
+      <param name="max_velocity_steps">${sts_max_velocity_steps}</param>
+      <param name="reset_states_on_activate">true</param>
+    </hardware>
+    <!-- Pan axis: rotates the payload around Z (Motor ID ${pan_motor_id}) -->
+    <joint name="pan_joint">
+      <param name="motor_id">${pan_motor_id}</param>
+      <param name="operating_mode">${pantilt_operating_mode}</param>
+      <param name="min_position">${pan_joint_lower}</param>
+      <param name="max_position">${pan_joint_upper}</param>
+      <param name="max_velocity">${max_velocity_rads}</param>
+      <param name="position_center_steps">2048</param>
+      <command_interface name="position"/>
+      <state_interface name="position"/>
+      <state_interface name="velocity"/>
+      <state_interface name="effort"/>
+      <state_interface name="voltage"/>
+      <state_interface name="temperature"/>
+      <state_interface name="current"/>
+      <state_interface name="is_moving"/>
+    </joint>
+    <!-- Tilt axis: rotates the payload around Y (Motor ID ${tilt_motor_id}) -->
+    <joint name="tilt_joint">
+      <param name="motor_id">${tilt_motor_id}</param>
+      <param name="operating_mode">${pantilt_operating_mode}</param>
+      <param name="min_position">${tilt_joint_lower}</param>
+      <param name="max_position">${tilt_joint_upper}</param>
+      <param name="max_velocity">${max_velocity_rads}</param>
+      <param name="position_center_steps">2048</param>
+      <command_interface name="position"/>
+      <state_interface name="position"/>
+      <state_interface name="velocity"/>
+      <state_interface name="effort"/>
+      <state_interface name="voltage"/>
+      <state_interface name="temperature"/>
+      <state_interface name="current"/>
+      <state_interface name="is_moving"/>
+    </joint>
+  </ros2_control>
 </robot>

File: lepantilt_description/urdf/pantilt.urdf (robot description, URDF)
Before this commit: robot lepantilt, 13 links, 12 joints
Links:
- removed link base_link
- removed link oak
- removed link oak_imu_frame
- removed link oak_left_camera_frame
- removed link oak_left_camera_optical_frame
- removed link oak_model_origin
- removed link oak_rgb_camera_frame
- removed link oak_rgb_camera_optical_frame
- removed link oak_right_camera_frame
- removed link oak_right_camera_optical_frame
- added link pantilt_base_link, mass 1.0; collision mesh filename=package://lepantilt_description/meshes/pantilt_base.stl; visual mesh filename=package://lepantilt_description/meshes/pan_motor.stl
- link pan_link: geometry collision mesh filename=package://lepantilt_description/meshes/pan_joint.stl; visual mesh filename=package://lepantilt_description/meshes/pan_joint.stl
- link tilt_link: geometry collision mesh filename=package://lepantilt_description/meshes/tilt_joint.stl; visual mesh filename=package://lepantilt_description/meshes/tilt_joint.stl
Joints:
- removed joint base_footprint_joint
- removed joint oak_imu_joint
- removed joint oak_left_camera_joint
- removed joint oak_left_camera_optical_joint
- removed joint oak_model_origin_joint
- removed joint oak_mount_joint
- removed joint oak_rgb_camera_joint
- removed joint oak_rgb_camera_optical_joint
- removed joint oak_right_camera_joint
- removed joint oak_right_camera_optical_joint
- added joint pantilt_mount_joint: type fixed, parent base_footprint, child pantilt_base_link, origin xyz=0 0 0 rpy=0 0 0
- joint pan_joint: parent base_link -> pantilt_base_link
- joint tilt_joint: limit lower=-1.5707963268 upper=1.5707963268 effort=2.942 velocity=5.21553467881118 -> lower=-1.5707963267948966 upper=1.5707963267948966 effort=2.942 velocity=5.21553467881118; origin xyz=0.0306 0 0.1025 rpy=-1.5707963268 1.5707963268 0 -> xyz=0.0306 0 0.1025 rpy=-1.5707963267948966 1.5707963267948966 0

File: lepantilt_description/urdf/pantilt.urdf.xacro (robot description, xacro)
@@ -3,180 +3,11 @@
   <xacro:include filename="$(find lepantilt_description)/urdf/pantilt.common.xacro"/>
   <xacro:include filename="$(find lepantilt_description)/urdf/pantilt.control.xacro"/>
+  <xacro:include filename="$(find lepantilt_description)/urdf/pantilt.module.xacro"/>
+  <!-- OAK-D camera and IMU integration -->
   <xacro:include filename="$(find depthai_descriptions)/urdf/include/depthai_macro.urdf.xacro"/>
-  <!-- Arguments (externally settable, default to property values in pantilt.control.xacro) -->
-  <xacro:arg name="serial_port"    default="${serial_port}"/>
-  <xacro:arg name="use_mock"       default="${use_mock}"/>
-  <xacro:arg name="use_sync_write" default="${use_sync_write}"/>
-  <material name="light_grey">
-    <color rgba="${light_grey_rgba}"/>
-  </material>
-  <material name="charcoal">
-    <color rgba="${charcoal_rgba}"/>
-  </material>
-  <!-- LINKS -->
-  <!-- Base footprint link (empty root — KDL does not support inertia on root link) -->
+  <!-- Standalone pantilt module instantiation -->
   <link name="base_footprint"/>
-  <!-- Base link -->
-  <link name="base_link">
-    <inertial>
-      <mass value="1.0"/>
-      <origin xyz="0 0 0" rpy="0 0 0"/>
-      <inertia ixx="0.01" ixy="0" ixz="0" iyy="0.01" iyz="0" izz="0.01"/>
-    </inertial>
-    <visual>
-      <origin xyz="0 0 0" rpy="0 0 ${pantilt_offset_rz}"/>
-      <geometry>
-        <mesh filename="package://lepantilt_description/meshes/pantilt_base.stl"/>
-      </geometry>
-      <material name="light_grey"/>
-    </visual>
-    <visual>
-      <origin xyz="0 0 0" rpy="0 0 ${pantilt_offset_rz}"/>
-      <geometry>
-        <mesh filename="package://lepantilt_description/meshes/pan_motor.stl"/>
-      </geometry>
-      <material name="charcoal"/>
-    </visual>
-    <collision>
-      <origin xyz="0 0 0" rpy="0 0 ${pantilt_offset_rz}"/>
-      <geometry>
-        <mesh filename="package://lepantilt_description/meshes/pantilt_base.stl"/>
-      </geometry>
-    </collision>
-  </link>
-  <!-- Pan link -->
-  <link name="pan_link">
-    <inertial>
-      <mass value="0.119226"/>
-      <origin xyz="-9.07886e-05 0.0590972 0.031089" rpy="0 0 0"/>
-      <inertia ixx="5.94278e-05" ixy="0" ixz="0" iyy="5.89975e-05" iyz="0" izz="3.13712e-05"/>
-    </inertial>
-    <visual>
-      <origin xyz="0 0 0" rpy="${pan_offset_rx} 0 ${pan_offset_rz}"/>
-      <geometry>
-        <mesh filename="package://lepantilt_description/meshes/pan_joint.stl"/>
-      </geometry>
-      <material name="light_grey"/>
-    </visual>
-    <visual>
-      <origin xyz="0 0 0" rpy="${pan_offset_rx} 0 ${pan_offset_rz}"/>
-      <geometry>
-        <mesh filename="package://lepantilt_description/meshes/tilt_motor.stl"/>
-      </geometry>
-      <material name="charcoal"/>
-    </visual>
-    <collision>
-      <origin xyz="0 0 0" rpy="${pan_offset_rx} 0 ${pan_offset_rz}"/>
-      <geometry>
-        <mesh filename="package://lepantilt_description/meshes/pan_joint.stl"/>
-      </geometry>
-    </collision>
-  </link>
-  <!-- Tilt link -->
-  <link name="tilt_link">
-    <inertial>
-      <mass value="0.1"/>
-      <origin xyz="0 0 0" rpy="0 0 0"/>
-      <inertia ixx="0.001" ixy="0" ixz="0" iyy="0.001" iyz="0" izz="0.001"/>
-    </inertial>
-    <visual>
-      <origin xyz="${tilt_visual_x} ${tilt_visual_y} ${tilt_visual_z}" rpy="${tilt_offset_rx} ${tilt_offset_ry} 0"/>
-      <geometry>
-        <mesh filename="package://lepantilt_description/meshes/tilt_joint.stl"/>
-      </geometry>
-      <material name="light_grey"/>
-    </visual>
-    <collision>
-      <origin xyz="${tilt_visual_x} ${tilt_visual_y} ${tilt_visual_z}" rpy="${tilt_offset_rx} ${tilt_offset_ry} 0"/>
-      <geometry>
-        <mesh filename="package://lepantilt_description/meshes/tilt_joint.stl"/>
-      </geometry>
-    </collision>
-  </link>
-  <!-- JOINTS -->
-  <!-- base_footprint fixed joint -->
-  <joint name="base_footprint_joint" type="fixed">
-    <parent link="base_footprint"/>
-    <child link="base_link"/>
-    <origin xyz="0 0 0" rpy="0 0 0"/>
-  </joint>
-  <!-- Pan joint (revolute) -->
-  <joint name="pan_joint" type="revolute">
-    <parent link="base_link"/>
-    <child link="pan_link"/>
-    <origin xyz="${pan_joint_x} 0 ${pan_joint_z}" rpy="0 0 0"/>
-    <axis xyz="0 0 1"/>
-    <limit lower="${pan_joint_lower}" upper="${pan_joint_upper}" effort="${max_torque_nm}" velocity="${max_velocity_rads}"/>
-  </joint>
-  <!-- Tilt joint (revolute) -->
-  <joint name="tilt_joint" type="revolute">
-    <parent link="pan_link"/>
-    <child link="tilt_link"/>
-    <origin xyz="${tilt_joint_x} 0 ${tilt_joint_z}" rpy="${tilt_joint_rx} ${tilt_joint_ry} 0"/>
-    <axis xyz="0 0 1"/>
-    <limit lower="${tilt_joint_lower}" upper="${tilt_joint_upper}" effort="${max_torque_nm}" velocity="${max_velocity_rads}"/>
-  </joint>
-  <!-- OAK-D-S2 camera (fixed to tilt_link via depthai_descriptions macro) -->
-  <xacro:depthai_camera
-    camera_name="oak"
-    camera_model="OAK-D-S2"
-    base_frame="oak"
-    parent="tilt_link"
-    cam_pos_x="${oak_pos_x}" cam_pos_y="${oak_pos_y}" cam_pos_z="0"
-    cam_roll="${oak_roll}" cam_pitch="0" cam_yaw="${oak_yaw}"
-    r="${charcoal_r}" g="${charcoal_g}" b="${charcoal_b}" a="${charcoal_a}"/>
-  <!-- OAK-D-S2 IMU frame -->
-  <link name="oak_imu_frame"/>
-  <joint name="oak_imu_joint" type="fixed">
-    <parent link="oak"/>
-    <child link="oak_imu_frame"/>
-    <origin xyz="${oak_imu_x} ${oak_imu_y} ${oak_imu_z}" rpy="${oak_imu_r} ${oak_imu_p} 0"/>
-  </joint>
-  <!-- ROS 2 CONTROL -->
-  <ros2_control name="lepantilt_control" type="system">
-    <hardware>
-      <plugin>sts_hardware_interface/STSHardwareInterface</plugin>
-      <param name="serial_port">$(arg serial_port)</param>
-      <param name="baud_rate">${baud_rate}</param>
-      <param name="communication_timeout_ms">100</param>
-      <param name="use_sync_write">$(arg use_sync_write)</param>
-      <param name="enable_mock_mode">$(arg use_mock)</param>
-      <param name="max_velocity_steps">${sts_max_velocity_steps}</param>
-      <param name="reset_states_on_activate">true</param>
-    </hardware>
-    <!-- Pan axis: rotates the payload around Z (Motor ID ${pan_motor_id}) -->
-    <joint name="pan_joint">
-      <param name="motor_id">${pan_motor_id}</param>
-      <param name="operating_mode">${pantilt_operating_mode}</param>
-      <param name="min_position">${pan_joint_lower}</param>
-      <param name="max_position">${pan_joint_upper}</param>
-      <param name="max_velocity">${max_velocity_rads}</param>
-      <param name="position_center_steps">2048</param>
-      <command_interface name="position"/>
-      <state_interface name="position"/>
-      <state_interface name="velocity"/>
-      <state_interface name="effort"/>
-      <state_interface name="voltage"/>
-      <state_interface name="temperature"/>
-      <state_interface name="current"/>
-      <state_interface name="is_moving"/>
-    </joint>
-    <!-- Tilt axis: rotates the payload around Y (Motor ID ${tilt_motor_id}) -->
-    <joint name="tilt_joint">
-      <param name="motor_id">${tilt_motor_id}</param>
-      <param name="operating_mode">${pantilt_operating_mode}</param>
-      <param name="min_position">${tilt_joint_lower}</param>
-      <param name="max_position">${tilt_joint_upper}</param>
-      <param name="max_velocity">${max_velocity_rads}</param>
-      <param name="position_center_steps">2048</param>
-      <command_interface name="position"/>
-      <state_interface name="position"/>
-      <state_interface name="velocity"/>
-      <state_interface name="effort"/>
-      <state_interface name="voltage"/>
-      <state_interface name="temperature"/>
-      <state_interface name="current"/>
-      <state_interface name="is_moving"/>
-    </joint>
-  </ros2_control>
+	<xacro:lepantilt_module parent="base_footprint">
+	  <origin xyz="0 0 0" rpy="0 0 0"/>
+	</xacro:lepantilt_module>
 </robot>
