Commit message: rename lepantilt to pantilt100

File: pt100_description/urdf/oakd_s2.urdf.xacro (robot description, xacro)
@@ -3,5 +3,5 @@
 	xmlns:xacro="http://ros.org/wiki/xacro">
 	<!--
-	  Custom OAK-D-S2 camera macro for lepantilt only.
+	  Custom OAK-D-S2 camera macro for pt100 only.
 	  This version allows direct color parameterization (r/g/b/a) for the mesh material.
 	-->
@@ -14,8 +14,8 @@
 		<!-- File prefix for mesh location -->
 		<xacro:if value="${simulation}">
-			<xacro:property name="mesh_path" value="file://$(find lepantilt_description)/meshes/oakd_s2.stl" />
+			<xacro:property name="mesh_path" value="file://$(find pt100_description)/meshes/oakd_s2.stl" />
 		</xacro:if>
 		<xacro:unless value="${simulation}">
-			<xacro:property name="mesh_path" value="package://lepantilt_description/meshes/oakd_s2.stl" />
+			<xacro:property name="mesh_path" value="package://pt100_description/meshes/oakd_s2.stl" />
 		</xacro:unless>
 		<!-- base_link of the sensor-->

File: pt100_description/urdf/pantilt.control.xacro (robot description, xacro)
@@ -22,5 +22,5 @@
   <xacro:property name="tilt_joint_upper" value="${pi/2}"/>
   <!-- ROS 2 CONTROL -->
-  <ros2_control name="lepantilt_control" type="system">
+  <ros2_control name="pt100_control" type="system">
     <hardware>
       <plugin>sts_hardware_interface/STSHardwareInterface</plugin>

File: pt100_description/urdf/pantilt.module.xacro (robot description, xacro)
@@ -1,6 +1,6 @@
 <?xml version="1.0"?>
 <robot xmlns:xacro="http://www.ros.org/wiki/xacro">
-  <xacro:include filename="$(find lepantilt_description)/urdf/pantilt.common.xacro"/>
-  <xacro:macro name="lepantilt_module" params="parent *origin">
+  <xacro:include filename="$(find pt100_description)/urdf/pantilt.common.xacro"/>
+  <xacro:macro name="pt100_module" params="parent *origin">
     <!-- Material definitions (referenced by links below) -->
     <material name="light_grey">
@@ -26,5 +26,5 @@
         <origin xyz="0 0 0" rpy="0 0 ${pantilt_offset_rz}"/>
         <geometry>
-          <mesh filename="package://lepantilt_description/meshes/pantilt_base.stl"/>
+          <mesh filename="package://pt100_description/meshes/pantilt_base.stl"/>
         </geometry>
         <material name="light_grey"/>
@@ -33,5 +33,5 @@
         <origin xyz="0 0 0" rpy="0 0 ${pantilt_offset_rz}"/>
         <geometry>
-          <mesh filename="package://lepantilt_description/meshes/pan_motor.stl"/>
+          <mesh filename="package://pt100_description/meshes/pan_motor.stl"/>
         </geometry>
         <material name="charcoal"/>
@@ -40,5 +40,5 @@
         <origin xyz="0 0 0" rpy="0 0 ${pantilt_offset_rz}"/>
         <geometry>
-          <mesh filename="package://lepantilt_description/meshes/pantilt_base.stl"/>
+          <mesh filename="package://pt100_description/meshes/pantilt_base.stl"/>
         </geometry>
       </collision>
@@ -54,5 +54,5 @@
         <origin xyz="0 0 0" rpy="${pan_offset_rx} 0 ${pan_offset_rz}"/>
         <geometry>
-          <mesh filename="package://lepantilt_description/meshes/pan_joint.stl"/>
+          <mesh filename="package://pt100_description/meshes/pan_joint.stl"/>
         </geometry>
         <material name="light_grey"/>
@@ -61,5 +61,5 @@
         <origin xyz="0 0 0" rpy="${pan_offset_rx} 0 ${pan_offset_rz}"/>
         <geometry>
-          <mesh filename="package://lepantilt_description/meshes/tilt_motor.stl"/>
+          <mesh filename="package://pt100_description/meshes/tilt_motor.stl"/>
         </geometry>
         <material name="charcoal"/>
@@ -68,5 +68,5 @@
         <origin xyz="0 0 0" rpy="${pan_offset_rx} 0 ${pan_offset_rz}"/>
         <geometry>
-          <mesh filename="package://lepantilt_description/meshes/pan_joint.stl"/>
+          <mesh filename="package://pt100_description/meshes/pan_joint.stl"/>
         </geometry>
       </collision>
@@ -82,5 +82,5 @@
         <origin xyz="${tilt_visual_x} ${tilt_visual_y} ${tilt_visual_z}" rpy="${tilt_offset_rx} ${tilt_offset_ry} 0"/>
         <geometry>
-          <mesh filename="package://lepantilt_description/meshes/tilt_joint.stl"/>
+          <mesh filename="package://pt100_description/meshes/tilt_joint.stl"/>
         </geometry>
         <material name="light_grey"/>
@@ -89,5 +89,5 @@
         <origin xyz="${tilt_visual_x} ${tilt_visual_y} ${tilt_visual_z}" rpy="${tilt_offset_rx} ${tilt_offset_ry} 0"/>
         <geometry>
-          <mesh filename="package://lepantilt_description/meshes/tilt_joint.stl"/>
+          <mesh filename="package://pt100_description/meshes/tilt_joint.stl"/>
         </geometry>
       </collision>
@@ -116,5 +116,5 @@
     </joint>
     <!-- OAK-D-S2 Camera + IMU -->
-    <xacro:include filename="$(find lepantilt_description)/urdf/oakd_s2.urdf.xacro"/>
+    <xacro:include filename="$(find pt100_description)/urdf/oakd_s2.urdf.xacro"/>
     <xacro:oakd_s2_camera
       camera_name="oak_link"

File: pt100_description/urdf/pantilt.urdf.xacro (robot description, xacro)
@@ -1,4 +1,4 @@
 <?xml version="1.0"?>
-<robot name="lepantilt" xmlns:xacro="http://www.ros.org/wiki/xacro">
+<robot name="pt100" xmlns:xacro="http://www.ros.org/wiki/xacro">
   <xacro:arg name="serial_port"    default="/dev/ttySERVO"/>
   <xacro:arg name="baud_rate"      default="1000000"/>
@@ -10,11 +10,11 @@
   <xacro:arg name="tilt_center_steps" default="2646"/>
   <xacro:arg name="pantilt_operating_mode" default="0"/>
-  <xacro:include filename="$(find lepantilt_description)/urdf/pantilt.common.xacro"/>
-  <xacro:include filename="$(find lepantilt_description)/urdf/pantilt.control.xacro"/>
-  <xacro:include filename="$(find lepantilt_description)/urdf/pantilt.module.xacro"/>
+  <xacro:include filename="$(find pt100_description)/urdf/pantilt.common.xacro"/>
+  <xacro:include filename="$(find pt100_description)/urdf/pantilt.control.xacro"/>
+  <xacro:include filename="$(find pt100_description)/urdf/pantilt.module.xacro"/>
   <!-- Standalone pantilt module instantiation -->
   <link name="base_footprint"/>
-	<xacro:lepantilt_module parent="base_footprint">
+	<xacro:pt100_module parent="base_footprint">
 	  <origin xyz="0 0 0" rpy="0 0 0"/>
-	</xacro:lepantilt_module>
+	</xacro:pt100_module>
 </robot>
