Commit message: update max speed and doc

File: pt100_description/urdf/pantilt.control.xacro (robot description, xacro)
@@ -13,5 +13,5 @@
   <xacro:property name="pantilt_operating_mode" default="0"/>  <!-- Position mode -->
   <xacro:property name="sts_max_velocity_steps" value="3400"/>  <!-- Max hardware velocity in steps/s (absolute motor limit, do not exceed) -->
-  <xacro:property name="max_velocity_steps" value="${int(sts_max_velocity_steps * 0.5)}"/> <!-- steps/second (85% of hardware max, 15% safety margin) -->
+  <xacro:property name="max_velocity_steps" value="${int(sts_max_velocity_steps * 0.85)}"/> <!-- steps/second (85% of hardware max, 15% safety margin) -->
   <xacro:property name="max_velocity_rads" value="${max_velocity_steps*2*pi/4096}"/> <!-- rad/s -->
   <xacro:property name="max_torque_nm" value="2.942"/>  <!-- N⋅m (30 kgf⋅cm for STS3215) -->
