Commit message: update tilt_joint stl and offsets

File: pt100_description/urdf/pantilt.common.xacro (robot description, xacro)
@@ -26,6 +26,6 @@
   <xacro:property name="tilt_visual_z" value="-0.0002"/>
   <!-- OAK-D-S2 camera mount offset (in tilt_link frame) -->
-  <xacro:property name="oak_pos_x" value="-0.03435"/>
-  <xacro:property name="oak_pos_y" value="-0.01"/>
+  <xacro:property name="oak_pos_x" value="-0.0306"/>
+  <xacro:property name="oak_pos_y" value="-0.012165"/>
   <!-- OAK-D-S2 camera mount orientation (in tilt_link frame) -->
   <xacro:property name="oak_roll" value="${-pi/2}"/>

File: pt100_description/urdf/pantilt.urdf (robot description, URDF)
Before this commit: robot pt100, 7 links, 6 joints
Joints:
- joint oak_link_center_joint: origin xyz=-0.03435 -0.01 0 rpy=-1.5707963267948966 0 -1.5707963267948966 -> xyz=-0.0306 -0.012165 0 rpy=-1.5707963267948966 0 -1.5707963267948966
