Commit message: Rename pt100-specific identifiers to pantilt, add pt101 mesh variant support
- Rename pt100.module.xacro/pt100_module, pt100_joints, pt100_control,
  and pt100_bringup/pt100.launch.py to their pantilt equivalents
- Add pantilt_config arg (pt100/pt101) to select mesh variants via
  pantilt.common.xacro; add pt101 pan_joint/pantilt_base meshes
- Rename pt100_description meshes for clarity:
  pantilt_base.stl -> pantilt_base_100.stl
  pan_joint.stl -> pan_joint_100.stl
  pan_joint_pt101.stl -> pan_joint_101.stl
  pantilt_base_pt101.stl -> pantilt_base_101.stl
  tilt_joint.stl -> tilt_joint_oakd_s2.stl
- Replace pantilt.urdf with generated pt100.urdf and pt101.urdf
  (relative ../meshes/ paths)
- Update README to match renamed files/macros

Co-Authored-By: Claude Sonnet 4.6 <noreply@anthropic.com>

File: pt100_description/urdf/pantilt.common.xacro (robot description, xacro)
@@ -5,4 +5,11 @@
   <xacro:property name="charcoal_rgba" value="0.15 0.15 0.15 1.0"/>
   <xacro:property name="charcoal_rgb" value="0.15"/>
+  <!-- Pan-tilt mechanical configuration: selects pantilt_base / pan_joint mesh
+       variants. "pt100" (default) uses the original meshes; "pt101" uses the
+       *_pt101 variants. All link/joint origins, axes, and the mount to the
+       host robot are shared and unchanged across configs — pt101 is a
+       drop-in mesh replacement only. -->
+  <xacro:arg name="pantilt_config" default="pt100"/>
+  <xacro:property name="pantilt_config" value="$(arg pantilt_config)"/>
   <!-- Pantilt base visual compensation / mount rotation (rad) -->
   <xacro:property name="pantilt_offset_rz" value="${pi/2}"/>
@@ -10,4 +17,39 @@
   <xacro:property name="pan_offset_rx" value="${pi/2}"/>
   <xacro:property name="pan_offset_rz" value="${pi/2}"/>
+  <xacro:property name="pantilt_base_mesh" value="pantilt_base_100.stl"/>
+  <xacro:property name="pan_joint_mesh" value="pan_joint_100.stl"/>
+  <!-- Mesh-local origin correction, applied to the body mesh of each link
+       only (not the motor meshes), in place of the shared
+       pantilt_offset_rz / pan_offset_rx+rz rotations above. pt100 meshes
+       reuse those shared rotations with zero translation (no-op). pt101
+       meshes need a different rotation (SO-ARM101's base_link/shoulder_link
+       frames are not simply Z-rotated copies of SO-ARM100's) plus a
+       translation; see derivation below. -->
+  <xacro:property name="pantilt_base_mesh_rpy" value="0 0 ${pantilt_offset_rz}"/>
+  <xacro:property name="pan_joint_mesh_rpy" value="${pan_offset_rx} 0 ${pan_offset_rz}"/>
+  <xacro:property name="pantilt_base_mesh_xyz" value="0 0 0"/>
+  <xacro:property name="pan_joint_mesh_xyz" value="0 0 0"/>
+  <xacro:if value="${pantilt_config == 'pt101'}">
+    <xacro:property name="pantilt_base_mesh" value="pantilt_base_101.stl"/>
+    <xacro:property name="pan_joint_mesh" value="pan_joint_101.stl"/>
+    <!-- pt101 meshes are pre-merged single-piece exports in their own native
+         frames (not aligned with pt100's). The rotation+translation below
+         was derived by matching each pt101 mesh's native bounding-box
+         extents/asymmetry against pt100's corresponding mesh's bounding box
+         after pt100's existing visual-compensation rotation
+         (pantilt_offset_rz for the base, pan_offset_rx+pan_offset_rz for the
+         pan body): pantilt_base_101.stl's bbox matches pantilt_base_100.stl's
+         (post-Rz(pi/2)) bbox after rotating by R(pi/2,0,pi/2); pan_joint_101.stl's
+         bbox matches pan_joint_100.stl's (post-R(pi/2,0,pi/2)) bbox after rotating
+         by R(pi/2,0,pi). The small translations align the base plate's
+         underside to Z=0 and the pan body's bbox to pt100's pan body bbox in
+         pan_link frame. Verified by rendering the full assembled chain
+         (base + pan_motor + pan body + tilt_motor + tilt body) for pt100 and
+         pt101 side by side from multiple angles. -->
+    <xacro:property name="pantilt_base_mesh_rpy" value="${pi/2} 0 ${pi/2}"/>
+    <xacro:property name="pan_joint_mesh_rpy" value="${pi/2} 0 ${pi}"/>
+    <xacro:property name="pantilt_base_mesh_xyz" value="0 0 0.0002"/>
+    <xacro:property name="pan_joint_mesh_xyz" value="-0.0120 0 -0.0002"/>
+  </xacro:if>
   <!-- Pan joint origin (in reoriented base_link frame) -->
   <xacro:property name="pan_joint_x" value="0.0452"/>

File: pt100_description/urdf/pantilt.control.xacro (robot description, xacro)
@@ -17,8 +17,8 @@
   <xacro:arg name="tilt_joint_upper"       default="1.5708"/>   <!-- rad, default +π/2 -->
   <!-- Hardware velocity ceiling — defined before <ros2_control> because the hardware
-       plugin param references it directly. pt100_joints receives the same value so
+       plugin param references it directly. pantilt_joints receives the same value so
        joint velocity limits stay consistent with what the interface is configured to enforce. -->
   <xacro:property name="sts_max_velocity_steps" value="$(arg sts_max_velocity_steps)"/>
-  <!-- Torque limit and joint limits as top-level properties — required by pt100.module.xacro
+  <!-- Torque limit and joint limits as top-level properties — required by pantilt.module.xacro
        for the URDF <limit> elements on the revolute joints. -->
   <xacro:property name="max_torque_nm"    value="2.942"/>  <!-- N⋅m (30 kgf⋅cm for STS3215) -->
@@ -29,5 +29,5 @@
   <xacro:include filename="$(find pt100_description)/urdf/pantilt.joints.xacro"/>
   <!-- ROS 2 CONTROL -->
-  <ros2_control name="pt100_control" type="system">
+  <ros2_control name="pantilt_control" type="system">
     <hardware>
       <plugin>sts_hardware_interface/STSHardwareInterface</plugin>
@@ -41,5 +41,5 @@
       <param name="reset_states_on_activate">true</param>
     </hardware>
-    <xacro:pt100_joints
+    <xacro:pantilt_joints
         pan_motor_id="$(arg pan_motor_id)"
         tilt_motor_id="$(arg tilt_motor_id)"

File: pt100_description/urdf/pantilt.joints.xacro (robot description, xacro)
@@ -2,5 +2,5 @@
 <robot xmlns:xacro="http://www.ros.org/wiki/xacro">
   <!--
-    pt100_joints macro — ros2_control joint declarations for the PT100 pan-tilt.
+    pantilt_joints macro — ros2_control joint declarations for the PT100 pan-tilt.
     Intended for embedding into a host robot's <ros2_control> block when the
     PT100 shares the host's serial bus (and therefore its hardware interface).
@@ -15,5 +15,5 @@
                                the value given to the hardware interface plugin
   -->
-  <xacro:macro name="pt100_joints" params="
+  <xacro:macro name="pantilt_joints" params="
       pan_motor_id:=1
       tilt_motor_id:=2
@@ -26,6 +26,6 @@
       tilt_joint_upper:=1.5708">
     <!-- 85% of hardware max — 15% safety margin; motor firmware handles profiling -->
-    <xacro:property name="pt100_max_velocity_steps" value="${int(sts_max_velocity_steps * 0.85)}"/>
-    <xacro:property name="pt100_max_velocity_rads"  value="${pt100_max_velocity_steps * 2 * pi / 4096}"/>
+    <xacro:property name="pantilt_max_velocity_steps" value="${int(sts_max_velocity_steps * 0.85)}"/>
+    <xacro:property name="pantilt_max_velocity_rads"  value="${pantilt_max_velocity_steps * 2 * pi / 4096}"/>
     <!-- Pan axis: rotates the payload around Z -->
     <joint name="pan_joint">
@@ -34,5 +34,5 @@
       <param name="min_position">${pan_joint_lower}</param>
       <param name="max_position">${pan_joint_upper}</param>
-      <param name="max_velocity">${pt100_max_velocity_rads}</param>
+      <param name="max_velocity">${pantilt_max_velocity_rads}</param>
       <param name="position_center_steps">${pan_center_steps}</param>
       <command_interface name="position"/>
@@ -51,5 +51,5 @@
       <param name="min_position">${tilt_joint_lower}</param>
       <param name="max_position">${tilt_joint_upper}</param>
-      <param name="max_velocity">${pt100_max_velocity_rads}</param>
+      <param name="max_velocity">${pantilt_max_velocity_rads}</param>
       <param name="position_center_steps">${tilt_center_steps}</param>
       <command_interface name="position"/>

File: pt100_description/urdf/pantilt.module.xacro (robot description, xacro)
@@ -3,5 +3,5 @@
   <xacro:include filename="$(find pt100_description)/urdf/pantilt.common.xacro"/>
   <xacro:include filename="$(find pt100_description)/urdf/oakd_s2.module.xacro"/>
-  <xacro:macro name="pt100_module" params="parent *origin">
+  <xacro:macro name="pantilt_module" params="parent *origin">
     <!-- Material definitions (referenced by links below) -->
     <material name="light_grey">
@@ -25,7 +25,7 @@
       </inertial>
       <visual>
-        <origin xyz="0 0 0" rpy="0 0 ${pantilt_offset_rz}"/>
+        <origin xyz="${pantilt_base_mesh_xyz}" rpy="${pantilt_base_mesh_rpy}"/>
         <geometry>
-          <mesh filename="package://pt100_description/meshes/pantilt_base.stl"/>
+          <mesh filename="package://pt100_description/meshes/${pantilt_base_mesh}"/>
         </geometry>
         <material name="light_grey"/>
@@ -39,7 +39,7 @@
       </visual>
       <collision>
-        <origin xyz="0 0 0" rpy="0 0 ${pantilt_offset_rz}"/>
+        <origin xyz="${pantilt_base_mesh_xyz}" rpy="${pantilt_base_mesh_rpy}"/>
         <geometry>
-          <mesh filename="package://pt100_description/meshes/pantilt_base.stl"/>
+          <mesh filename="package://pt100_description/meshes/${pantilt_base_mesh}"/>
         </geometry>
       </collision>
@@ -53,7 +53,7 @@
       </inertial>
       <visual>
-        <origin xyz="0 0 0" rpy="${pan_offset_rx} 0 ${pan_offset_rz}"/>
+        <origin xyz="${pan_joint_mesh_xyz}" rpy="${pan_joint_mesh_rpy}"/>
         <geometry>
-          <mesh filename="package://pt100_description/meshes/pan_joint.stl"/>
+          <mesh filename="package://pt100_description/meshes/${pan_joint_mesh}"/>
         </geometry>
         <material name="light_grey"/>
@@ -67,7 +67,7 @@
       </visual>
       <collision>
-        <origin xyz="0 0 0" rpy="${pan_offset_rx} 0 ${pan_offset_rz}"/>
+        <origin xyz="${pan_joint_mesh_xyz}" rpy="${pan_joint_mesh_rpy}"/>
         <geometry>
-          <mesh filename="package://pt100_description/meshes/pan_joint.stl"/>
+          <mesh filename="package://pt100_description/meshes/${pan_joint_mesh}"/>
         </geometry>
       </collision>
@@ -83,5 +83,5 @@
         <origin xyz="${tilt_visual_x} ${tilt_visual_y} ${tilt_visual_z}" rpy="${tilt_offset_rx} ${tilt_offset_ry} 0"/>
         <geometry>
-          <mesh filename="package://pt100_description/meshes/tilt_joint.stl"/>
+          <mesh filename="package://pt100_description/meshes/tilt_joint_oakd_s2.stl"/>
         </geometry>
         <material name="light_grey"/>
@@ -90,5 +90,5 @@
         <origin xyz="${tilt_visual_x} ${tilt_visual_y} ${tilt_visual_z}" rpy="${tilt_offset_rx} ${tilt_offset_ry} 0"/>
         <geometry>
-          <mesh filename="package://pt100_description/meshes/tilt_joint.stl"/>
+          <mesh filename="package://pt100_description/meshes/tilt_joint_oakd_s2.stl"/>
         </geometry>
       </collision>

File: pt100_description/urdf/pantilt.urdf.xacro (robot description, xacro)
@@ -1,4 +1,4 @@
 <?xml version="1.0"?>
-<robot name="pt100" xmlns:xacro="http://www.ros.org/wiki/xacro">
+<robot name="pantilt" xmlns:xacro="http://www.ros.org/wiki/xacro">
   <xacro:arg name="serial_port"    default="/dev/ttySERVO"/>
   <xacro:arg name="baud_rate"      default="1000000"/>
@@ -11,9 +11,9 @@
   <xacro:include filename="$(find pt100_description)/urdf/pantilt.common.xacro"/>
   <xacro:include filename="$(find pt100_description)/urdf/pantilt.control.xacro"/>
-  <xacro:include filename="$(find pt100_description)/urdf/pt100.module.xacro"/>
+  <xacro:include filename="$(find pt100_description)/urdf/pantilt.module.xacro"/>
   <!-- Standalone pantilt module instantiation -->
   <link name="base_footprint"/>
-	<xacro:pt100_module parent="base_footprint">
+	<xacro:pantilt_module parent="base_footprint">
 	  <origin xyz="0 0 0" rpy="0 0 0"/>
-	</xacro:pt100_module>
+	</xacro:pantilt_module>
 </robot>

File: pt100_description/urdf/pt100.urdf (robot description, URDF)
Before this commit: robot pt100, 7 links, 6 joints
Links:
- link pan_link: geometry collision mesh filename=../meshes/pan_joint_100.stl; visual mesh filename=../meshes/pan_joint_100.stl
- link pantilt_base_link: geometry collision mesh filename=../meshes/pantilt_base_100.stl; visual mesh filename=../meshes/pan_motor.stl
- link tilt_link: geometry collision mesh filename=../meshes/tilt_joint_oakd_s2.stl; visual mesh filename=../meshes/tilt_joint_oakd_s2.stl
