Commit message: refactor: rename pt100_description/pt100_control/pt100_bringup to pt_description/pt_control/pt_bringup
Drops the redundant "100" suffix from package names since pantilt_config
already selects between pt100/pt101 mesh variants at the URDF level.

File: pt_description/urdf/oakd_s2.module.xacro (robot description, xacro)
@@ -14,8 +14,8 @@
 		<!-- File prefix for mesh location -->
 		<xacro:if value="${simulation}">
-			<xacro:property name="mesh_path" value="file://$(find pt100_description)/meshes/oakd_s2.stl" />
+			<xacro:property name="mesh_path" value="file://$(find pt_description)/meshes/oakd_s2.stl" />
 		</xacro:if>
 		<xacro:unless value="${simulation}">
-			<xacro:property name="mesh_path" value="package://pt100_description/meshes/oakd_s2.stl" />
+			<xacro:property name="mesh_path" value="package://pt_description/meshes/oakd_s2.stl" />
 		</xacro:unless>
 		<!-- base_link of the sensor-->

File: pt_description/urdf/pantilt.control.xacro (robot description, xacro)
@@ -27,5 +27,5 @@
   <xacro:property name="tilt_joint_lower" value="$(arg tilt_joint_lower)"/>
   <xacro:property name="tilt_joint_upper" value="$(arg tilt_joint_upper)"/>
-  <xacro:include filename="$(find pt100_description)/urdf/pantilt.joints.xacro"/>
+  <xacro:include filename="$(find pt_description)/urdf/pantilt.joints.xacro"/>
   <!-- ROS 2 CONTROL -->
   <ros2_control name="pantilt_control" type="system">

File: pt_description/urdf/pantilt.module.xacro (robot description, xacro)
@@ -1,6 +1,6 @@
 <?xml version="1.0"?>
 <robot xmlns:xacro="http://www.ros.org/wiki/xacro">
-  <xacro:include filename="$(find pt100_description)/urdf/pantilt.common.xacro"/>
-  <xacro:include filename="$(find pt100_description)/urdf/oakd_s2.module.xacro"/>
+  <xacro:include filename="$(find pt_description)/urdf/pantilt.common.xacro"/>
+  <xacro:include filename="$(find pt_description)/urdf/oakd_s2.module.xacro"/>
   <xacro:macro name="pantilt_module" params="parent *origin">
     <!-- Material definitions (referenced by links below) -->
@@ -27,5 +27,5 @@
         <origin xyz="${pantilt_base_mesh_xyz}" rpy="${pantilt_base_mesh_rpy}"/>
         <geometry>
-          <mesh filename="package://pt100_description/meshes/${pantilt_base_mesh}"/>
+          <mesh filename="package://pt_description/meshes/${pantilt_base_mesh}"/>
         </geometry>
         <material name="light_grey"/>
@@ -34,5 +34,5 @@
         <origin xyz="0 0 0" rpy="0 0 ${pantilt_offset_rz}"/>
         <geometry>
-          <mesh filename="package://pt100_description/meshes/pan_motor.stl"/>
+          <mesh filename="package://pt_description/meshes/pan_motor.stl"/>
         </geometry>
         <material name="charcoal"/>
@@ -41,5 +41,5 @@
         <origin xyz="${pantilt_base_mesh_xyz}" rpy="${pantilt_base_mesh_rpy}"/>
         <geometry>
-          <mesh filename="package://pt100_description/meshes/${pantilt_base_mesh}"/>
+          <mesh filename="package://pt_description/meshes/${pantilt_base_mesh}"/>
         </geometry>
       </collision>
@@ -55,5 +55,5 @@
         <origin xyz="${pan_joint_mesh_xyz}" rpy="${pan_joint_mesh_rpy}"/>
         <geometry>
-          <mesh filename="package://pt100_description/meshes/${pan_joint_mesh}"/>
+          <mesh filename="package://pt_description/meshes/${pan_joint_mesh}"/>
         </geometry>
         <material name="light_grey"/>
@@ -62,5 +62,5 @@
         <origin xyz="0 0 0" rpy="${pan_offset_rx} 0 ${pan_offset_rz}"/>
         <geometry>
-          <mesh filename="package://pt100_description/meshes/tilt_motor.stl"/>
+          <mesh filename="package://pt_description/meshes/tilt_motor.stl"/>
         </geometry>
         <material name="charcoal"/>
@@ -69,5 +69,5 @@
         <origin xyz="${pan_joint_mesh_xyz}" rpy="${pan_joint_mesh_rpy}"/>
         <geometry>
-          <mesh filename="package://pt100_description/meshes/${pan_joint_mesh}"/>
+          <mesh filename="package://pt_description/meshes/${pan_joint_mesh}"/>
         </geometry>
       </collision>
@@ -83,5 +83,5 @@
         <origin xyz="${tilt_visual_x} ${tilt_visual_y} ${tilt_visual_z}" rpy="${tilt_offset_rx} ${tilt_offset_ry} 0"/>
         <geometry>
-          <mesh filename="package://pt100_description/meshes/tilt_joint_oakd_s2.stl"/>
+          <mesh filename="package://pt_description/meshes/tilt_joint_oakd_s2.stl"/>
         </geometry>
         <material name="light_grey"/>
@@ -90,5 +90,5 @@
         <origin xyz="${tilt_visual_x} ${tilt_visual_y} ${tilt_visual_z}" rpy="${tilt_offset_rx} ${tilt_offset_ry} 0"/>
         <geometry>
-          <mesh filename="package://pt100_description/meshes/tilt_joint_oakd_s2.stl"/>
+          <mesh filename="package://pt_description/meshes/tilt_joint_oakd_s2.stl"/>
         </geometry>
       </collision>

File: pt_description/urdf/pantilt.urdf.xacro (robot description, xacro)
@@ -9,7 +9,7 @@
   <xacro:arg name="pan_center_steps" default="2048"/>
   <xacro:arg name="tilt_center_steps" default="2646"/>
-  <xacro:include filename="$(find pt100_description)/urdf/pantilt.common.xacro"/>
-  <xacro:include filename="$(find pt100_description)/urdf/pantilt.control.xacro"/>
-  <xacro:include filename="$(find pt100_description)/urdf/pantilt.module.xacro"/>
+  <xacro:include filename="$(find pt_description)/urdf/pantilt.common.xacro"/>
+  <xacro:include filename="$(find pt_description)/urdf/pantilt.control.xacro"/>
+  <xacro:include filename="$(find pt_description)/urdf/pantilt.module.xacro"/>
   <!-- Standalone pantilt module instantiation -->
   <link name="base_footprint"/>
