Commit message: Strip MuJoCo/OAK-D VIO stack for RosCon UK 2026 demo
Removes MuJoCo simulation support (mjcf assets, mujoco_ros2_control_plugins.yaml,
ros2_control_hardware_type mujoco/gazebo branching in pantilt.control.xacro/
pantilt.module.xacro/pantilt.joints.xacro) and the OAK-D VIO/octomap/
depthimage_to_laserscan/pcl_compressor_node pipeline (oakd.launch.py and its configs),
consolidating back to real-hardware-only for this demo branch.

Co-Authored-By: Claude Sonnet 5 <noreply@anthropic.com>

File: pt_description/urdf/oakd_s2.module.xacro (robot description, xacro)
@@ -1,8 +1,9 @@
 <?xml version="1.0"?>
-<robot name="depthai_camera"
+<robot name="oakd_s2_mount"
 	xmlns:xacro="http://ros.org/wiki/xacro">
 	<!--
-	  Custom OAK-D-S2 camera macro, shared by both pt100/pt101.
-	  This version allows direct color parameterization (r/g/b/a) for the mesh material.
+	  OAK-D-S2 mount macro, shared by both pt100/pt101: mesh, link, and fixed joints only
+	  (TF/visual geometry) - no camera driver, sensor, or ROS interface. This version
+	  allows direct color parameterization (r/g/b/a) for the mesh material.
 	-->
 	<xacro:macro name="oakd_s2_camera"
@@ -10,13 +11,7 @@
 											   cam_pos_x cam_pos_y cam_pos_z
 											   cam_roll cam_pitch cam_yaw
-											   r:=0.1 g:=0.1 b:=0.1 a:=1.0 simulation:=false
+											   r:=0.1 g:=0.1 b:=0.1 a:=1.0
 											   imu_frame:=oak_imu_frame">
-		<!-- File prefix for mesh location -->
-		<xacro:if value="${simulation}">
-			<xacro:property name="mesh_path" value="file://$(find pt_description)/meshes/oakd_s2.stl" />
-		</xacro:if>
-		<xacro:unless value="${simulation}">
-			<xacro:property name="mesh_path" value="package://pt_description/meshes/oakd_s2.stl" />
-		</xacro:unless>
+		<xacro:property name="mesh_path" value="package://pt_description/meshes/oakd_s2.stl" />
 		<!-- base_link of the sensor-->
 		<link name="${base_frame}" />

File: pt_description/urdf/pantilt.control.xacro (robot description, xacro)
@@ -16,20 +16,4 @@
   <xacro:arg name="tilt_joint_lower"       default="-1.5708"/>  <!-- rad, default -π/2 -->
   <xacro:arg name="tilt_joint_upper"       default="1.5708"/>   <!-- rad, default +π/2 -->
-  <!-- Simulation -->
-  <!-- "real" (default) keeps the STS3215 serial hardware plugin below unchanged.
-       "gazebo" swaps the <hardware> plugin for gz_ros2_control/GazeboSimSystem.
-       "mujoco" swaps it for mujoco_ros2_control/MujocoSystemInterface.
-       Both implement the same SystemInterface contract - the joints and controllers stay
-       identical in all three cases. -->
-  <xacro:arg name="ros2_control_hardware_type" default="real"/>
-  <!-- Path to the controllers YAML the embedded controller_manager should load; only
-       used when the <gazebo> plugin below is actually instantiated (i.e. in sim). -->
-  <xacro:arg name="simulation_controllers" default=""/>
-  <!-- mujoco mode only: path to the xacro-generated MJCF scene (pt_description/mjcf/
-       pantilt.mjcf.xacro, xacro-processed at launch time with pantilt_config picking the
-       pt100/pt101 mesh variant - see pt_control/launch/pantilt.launch.py) and whether to
-       open the MuJoCo Simulate viewer window. -->
-  <xacro:arg name="mujoco_model" default=""/>
-  <xacro:arg name="mujoco_headless" default="false"/>
   <!-- Hardware velocity ceiling — defined before <ros2_control> because the hardware
        plugin param references it directly. pantilt_joints receives the same value so
@@ -39,6 +23,7 @@
        pantilt.module.xacro for the URDF <limit> elements on the revolute joints.
        pantilt_max_velocity_rads duplicates pantilt_joints' own local computation
-       (pantilt.joints.xacro) - only used by module.xacro's gazebo-mode <limit velocity>,
-       real mode keeps velocity="1e6" (see module.xacro's comment on why) regardless. -->
+       (pantilt.joints.xacro) - unused by module.xacro's <limit velocity> itself (that stays
+       at velocity="1e6", see module.xacro's comment on why), kept for the max_velocity
+       <param> passed into pantilt_joints below. -->
   <!-- This project runs the 12V STS3215 variant: 30 kgf*cm stall torque per Feetech's
        datasheet for that voltage option (not the 7.4V/19.5 kgf*cm variant used by stock
@@ -55,23 +40,13 @@
   <ros2_control name="pantilt_control" type="system">
     <hardware>
-      <xacro:if value="${'$(arg ros2_control_hardware_type)' == 'gazebo'}">
-        <plugin>gz_ros2_control/GazeboSimSystem</plugin>
-      </xacro:if>
-      <xacro:if value="${'$(arg ros2_control_hardware_type)' == 'mujoco'}">
-        <plugin>mujoco_ros2_control/MujocoSystemInterface</plugin>
-        <param name="mujoco_model">$(arg mujoco_model)</param>
-        <param name="headless">$(arg mujoco_headless)</param>
-      </xacro:if>
-      <xacro:if value="${'$(arg ros2_control_hardware_type)' == 'real'}">
-        <plugin>sts_hardware_interface/STSHardwareInterface</plugin>
-        <param name="serial_port">$(arg serial_port)</param>
-        <param name="baud_rate">$(arg baud_rate)</param>
-        <param name="communication_timeout_ms">100</param>
-        <param name="use_sync_write">$(arg use_sync_write)</param>
-        <param name="enable_mock_mode">$(arg use_mock)</param>
-        <param name="max_velocity_steps">${sts_max_velocity_steps}</param>
-        <param name="proportional_vel_max">$(arg proportional_vel_max)</param>
-        <param name="reset_states_on_activate">true</param>
-      </xacro:if>
+      <plugin>sts_hardware_interface/STSHardwareInterface</plugin>
+      <param name="serial_port">$(arg serial_port)</param>
+      <param name="baud_rate">$(arg baud_rate)</param>
+      <param name="communication_timeout_ms">100</param>
+      <param name="use_sync_write">$(arg use_sync_write)</param>
+      <param name="enable_mock_mode">$(arg use_mock)</param>
+      <param name="max_velocity_steps">${sts_max_velocity_steps}</param>
+      <param name="proportional_vel_max">$(arg proportional_vel_max)</param>
+      <param name="reset_states_on_activate">true</param>
     </hardware>
     <xacro:pantilt_joints
@@ -84,6 +59,5 @@
         pan_joint_upper="${pan_joint_upper}"
         tilt_joint_lower="${tilt_joint_lower}"
-        tilt_joint_upper="${tilt_joint_upper}"
-        ros2_control_hardware_type="$(arg ros2_control_hardware_type)"/>
+        tilt_joint_upper="${tilt_joint_upper}"/>
   </ros2_control>
 </robot>

File: pt_description/urdf/pantilt.joints.xacro (robot description, xacro)
@@ -24,6 +24,5 @@
       pan_joint_upper:=1.5708
       tilt_joint_lower:=-1.5708
-      tilt_joint_upper:=1.5708
-      ros2_control_hardware_type:=real">
+      tilt_joint_upper:=1.5708">
     <!-- 85% of hardware max — 15% safety margin; motor firmware handles profiling -->
     <xacro:property name="pantilt_max_velocity_steps" value="${int(sts_max_velocity_steps * 0.85)}"/>
@@ -41,13 +40,8 @@
       <state_interface name="velocity"/>
       <state_interface name="effort"/>
-      <!-- Real-hardware-only telemetry: neither gz_ros2_control/GazeboSimSystem nor
-           mujoco_ros2_control/MujocoSystemInterface know position/velocity/effort-only
-           joints, and simulated joints have no real telemetry for these. -->
-      <xacro:if value="${ros2_control_hardware_type == 'real'}">
-        <state_interface name="voltage"/>
-        <state_interface name="temperature"/>
-        <state_interface name="current"/>
-        <state_interface name="is_moving"/>
-      </xacro:if>
+      <state_interface name="voltage"/>
+      <state_interface name="temperature"/>
+      <state_interface name="current"/>
+      <state_interface name="is_moving"/>
     </joint>
     <!-- Tilt axis: rotates the payload around Y -->
@@ -63,13 +57,8 @@
       <state_interface name="velocity"/>
       <state_interface name="effort"/>
-      <!-- Real-hardware-only telemetry: neither gz_ros2_control/GazeboSimSystem nor
-           mujoco_ros2_control/MujocoSystemInterface know position/velocity/effort-only
-           joints, and simulated joints have no real telemetry for these. -->
-      <xacro:if value="${ros2_control_hardware_type == 'real'}">
-        <state_interface name="voltage"/>
-        <state_interface name="temperature"/>
-        <state_interface name="current"/>
-        <state_interface name="is_moving"/>
-      </xacro:if>
+      <state_interface name="voltage"/>
+      <state_interface name="temperature"/>
+      <state_interface name="current"/>
+      <state_interface name="is_moving"/>
     </joint>
   </xacro:macro>

File: pt_description/urdf/pantilt.module.xacro (robot description, xacro)
@@ -94,8 +94,7 @@
       </collision>
     </link>
-    <!-- real mode: velocity="1e6" (unreachable) disables JointSaturationLimiter's clipping,
-         since joy_teleop's absolute position jumps would otherwise trip spurious limit
-         errors. gazebo mode: uses the real computed ceiling instead, since GazeboSimSystem
-         actually enforces this limit on the simulated joint. -->
+    <!-- velocity="1e6" (unreachable) disables JointSaturationLimiter's clipping, since
+         joy_teleop's absolute position jumps would otherwise trip spurious limit errors.
+         The real speed ceiling comes from max_velocity in the <ros2_control> block. -->
     <!-- Pan joint (revolute) -->
     <joint name="pan_joint" type="revolute">
@@ -104,5 +103,5 @@
       <origin xyz="${pan_joint_x} 0 ${pan_joint_z}" rpy="0 0 0"/>
       <axis xyz="0 0 1"/>
-      <limit lower="${pan_joint_lower}" upper="${pan_joint_upper}" effort="${max_torque_nm}" velocity="${1e6 if '$(arg ros2_control_hardware_type)' == 'real' else pantilt_max_velocity_rads}"/>
+      <limit lower="${pan_joint_lower}" upper="${pan_joint_upper}" effort="${max_torque_nm}" velocity="1e6"/>
     </joint>
     <!-- Tilt joint (revolute) -->
@@ -112,5 +111,5 @@
       <origin xyz="${tilt_joint_x} 0 ${tilt_joint_z}" rpy="${tilt_joint_rx} ${tilt_joint_ry} 0"/>
       <axis xyz="0 0 -1"/>
-      <limit lower="${tilt_joint_lower}" upper="${tilt_joint_upper}" effort="${max_torque_nm}" velocity="${1e6 if '$(arg ros2_control_hardware_type)' == 'real' else pantilt_max_velocity_rads}"/>
+      <limit lower="${tilt_joint_lower}" upper="${tilt_joint_upper}" effort="${max_torque_nm}" velocity="1e6"/>
     </joint>
     <!-- OAK-D-S2 Camera + IMU -->

File: pt_description/urdf/pantilt.urdf.xacro (robot description, xacro)
@@ -17,11 +17,3 @@
 	  <origin xyz="0 0 0" rpy="0 0 0"/>
 	</xacro:pantilt_module>
-  <!-- Gazebo simulation: spawns controller_manager inside the gz_sim process, loading
-       $(arg simulation_controllers). Inert (ignored) outside Gazebo, so this is safe to
-       leave in place regardless of ros2_control_hardware_type. -->
-  <gazebo>
-    <plugin filename="gz_ros2_control-system" name="gz_ros2_control::GazeboSimROS2ControlPlugin">
-      <parameters>$(arg simulation_controllers)</parameters>
-    </plugin>
-  </gazebo>
 </robot>

File: pt_description/urdf/pt100.urdf (robot description, URDF)
Before this commit: robot pantilt, 7 links, 6 joints
Joints:
- joint pan_joint: limit lower=-1.5708 upper=1.5708 effort=2.942 velocity=1000000.0 -> lower=-1.5708 upper=1.5708 effort=2.942 velocity=1e6
- joint tilt_joint: limit lower=-1.5708 upper=1.5708 effort=2.942 velocity=1000000.0 -> lower=-1.5708 upper=1.5708 effort=2.942 velocity=1e6

File: pt_description/urdf/pt101.urdf (robot description, URDF)
Before this commit: robot pantilt, 7 links, 6 joints
Joints:
- joint pan_joint: limit lower=-1.5708 upper=1.5708 effort=2.942 velocity=1000000.0 -> lower=-1.5708 upper=1.5708 effort=2.942 velocity=1e6
- joint tilt_joint: limit lower=-1.5708 upper=1.5708 effort=2.942 velocity=1000000.0 -> lower=-1.5708 upper=1.5708 effort=2.942 velocity=1e6
