Commit message: Add gz_ros2_control support for Gazebo simulation
pantilt.control.xacro/pantilt.joints.xacro: ros2_control_hardware_type
("real"/"gazebo") swaps the <hardware> plugin between STSHardwareInterface and
gz_ros2_control/GazeboSimSystem, and drops the STS-specific telemetry state
interfaces (voltage/temperature/current/is_moving) that GazeboSimSystem can't
back with simulated data.

pantilt.module.xacro: the pan/tilt joints' velocity="1e6" limit (deliberately
unbounded on real hardware, since the STS firmware does its own velocity
profiling) now uses the real computed velocity ceiling in gazebo mode instead,
where GazeboSimSystem has no hardware profiling to defer to and would
otherwise let the joint snap to its target instantly.

pantilt.urdf.xacro: adds the <gazebo> plugin block that spawns
controller_manager embedded inside gz_sim, loading simulation_controllers.

pt_control/pt_bringup pantilt.launch.py: thread ros2_control_hardware_type
through, skip the standalone controller_manager in gazebo mode (gz_sim's
embedded one takes over), and pt_bringup gains sim/gui args that start Gazebo
+ bridge /clock + spawn the entity instead of the real oakd camera driver.

All of this is inert outside Gazebo - real-hardware xacro output and launch
behavior are unchanged.

Co-Authored-By: Claude Sonnet 5 <noreply@anthropic.com>

File: pt_description/urdf/pantilt.control.xacro (robot description, xacro)
@@ -16,11 +16,25 @@
   <xacro:arg name="tilt_joint_lower"       default="-1.5708"/>  <!-- rad, default -π/2 -->
   <xacro:arg name="tilt_joint_upper"       default="1.5708"/>   <!-- rad, default +π/2 -->
+  <!-- Gazebo simulation -->
+  <!-- "real" (default) keeps the STS3215 serial hardware plugin below unchanged.
+       "gazebo" swaps the <hardware> plugin for gz_ros2_control/GazeboSimSystem, which
+       implements the same SystemInterface contract - the joints and controllers stay
+       identical either way. -->
+  <xacro:arg name="ros2_control_hardware_type" default="real"/>
+  <!-- Path to the controllers YAML the embedded controller_manager should load; only
+       used when the <gazebo> plugin below is actually instantiated (i.e. in sim). -->
+  <xacro:arg name="simulation_controllers" default=""/>
   <!-- Hardware velocity ceiling — defined before <ros2_control> because the hardware
        plugin param references it directly. pantilt_joints receives the same value so
        joint velocity limits stay consistent with what the interface is configured to enforce. -->
   <xacro:property name="sts_max_velocity_steps" value="$(arg sts_max_velocity_steps)"/>
-  <!-- Torque limit and joint limits as top-level properties — required by pantilt.module.xacro
-       for the URDF <limit> elements on the revolute joints. -->
+  <!-- Torque/velocity limits and joint limits as top-level properties — required by
+       pantilt.module.xacro for the URDF <limit> elements on the revolute joints.
+       pantilt_max_velocity_rads duplicates pantilt_joints' own local computation
+       (pantilt.joints.xacro) - only used by module.xacro's gazebo-mode <limit velocity>,
+       real mode keeps velocity="1e6" (see module.xacro's comment on why) regardless. -->
   <xacro:property name="max_torque_nm"    value="2.942"/>  <!-- N⋅m (30 kgf⋅cm for STS3215) -->
+  <xacro:property name="pantilt_max_velocity_steps" value="${int(sts_max_velocity_steps * 0.85)}"/>
+  <xacro:property name="pantilt_max_velocity_rads"  value="${pantilt_max_velocity_steps * 2 * pi / 4096}"/>
   <xacro:property name="pan_joint_lower"  value="$(arg pan_joint_lower)"/>
   <xacro:property name="pan_joint_upper"  value="$(arg pan_joint_upper)"/>
@@ -31,13 +45,18 @@
   <ros2_control name="pantilt_control" type="system">
     <hardware>
-      <plugin>sts_hardware_interface/STSHardwareInterface</plugin>
-      <param name="serial_port">$(arg serial_port)</param>
-      <param name="baud_rate">$(arg baud_rate)</param>
-      <param name="communication_timeout_ms">100</param>
-      <param name="use_sync_write">$(arg use_sync_write)</param>
-      <param name="enable_mock_mode">$(arg use_mock)</param>
-      <param name="max_velocity_steps">${sts_max_velocity_steps}</param>
-      <param name="proportional_vel_max">$(arg proportional_vel_max)</param>
-      <param name="reset_states_on_activate">true</param>
+      <xacro:if value="${'$(arg ros2_control_hardware_type)' == 'gazebo'}">
+        <plugin>gz_ros2_control/GazeboSimSystem</plugin>
+      </xacro:if>
+      <xacro:unless value="${'$(arg ros2_control_hardware_type)' == 'gazebo'}">
+        <plugin>sts_hardware_interface/STSHardwareInterface</plugin>
+        <param name="serial_port">$(arg serial_port)</param>
+        <param name="baud_rate">$(arg baud_rate)</param>
+        <param name="communication_timeout_ms">100</param>
+        <param name="use_sync_write">$(arg use_sync_write)</param>
+        <param name="enable_mock_mode">$(arg use_mock)</param>
+        <param name="max_velocity_steps">${sts_max_velocity_steps}</param>
+        <param name="proportional_vel_max">$(arg proportional_vel_max)</param>
+        <param name="reset_states_on_activate">true</param>
+      </xacro:unless>
     </hardware>
     <xacro:pantilt_joints
@@ -50,5 +69,6 @@
         pan_joint_upper="${pan_joint_upper}"
         tilt_joint_lower="${tilt_joint_lower}"
-        tilt_joint_upper="${tilt_joint_upper}"/>
+        tilt_joint_upper="${tilt_joint_upper}"
+        ros2_control_hardware_type="$(arg ros2_control_hardware_type)"/>
   </ros2_control>
 </robot>

File: pt_description/urdf/pantilt.joints.xacro (robot description, xacro)
@@ -24,5 +24,6 @@
       pan_joint_upper:=1.5708
       tilt_joint_lower:=-1.5708
-      tilt_joint_upper:=1.5708">
+      tilt_joint_upper:=1.5708
+      ros2_control_hardware_type:=real">
     <!-- 85% of hardware max — 15% safety margin; motor firmware handles profiling -->
     <xacro:property name="pantilt_max_velocity_steps" value="${int(sts_max_velocity_steps * 0.85)}"/>
@@ -40,8 +41,12 @@
       <state_interface name="velocity"/>
       <state_interface name="effort"/>
-      <state_interface name="voltage"/>
-      <state_interface name="temperature"/>
-      <state_interface name="current"/>
-      <state_interface name="is_moving"/>
+      <!-- Real-hardware-only telemetry: gz_ros2_control/GazeboSimSystem only knows
+           position/velocity/effort, and simulated joints have no real telemetry for these. -->
+      <xacro:unless value="${ros2_control_hardware_type == 'gazebo'}">
+        <state_interface name="voltage"/>
+        <state_interface name="temperature"/>
+        <state_interface name="current"/>
+        <state_interface name="is_moving"/>
+      </xacro:unless>
     </joint>
     <!-- Tilt axis: rotates the payload around Y -->
@@ -57,8 +62,12 @@
       <state_interface name="velocity"/>
       <state_interface name="effort"/>
-      <state_interface name="voltage"/>
-      <state_interface name="temperature"/>
-      <state_interface name="current"/>
-      <state_interface name="is_moving"/>
+      <!-- Real-hardware-only telemetry: gz_ros2_control/GazeboSimSystem only knows
+           position/velocity/effort, and simulated joints have no real telemetry for these. -->
+      <xacro:unless value="${ros2_control_hardware_type == 'gazebo'}">
+        <state_interface name="voltage"/>
+        <state_interface name="temperature"/>
+        <state_interface name="current"/>
+        <state_interface name="is_moving"/>
+      </xacro:unless>
     </joint>
   </xacro:macro>

File: pt_description/urdf/pantilt.module.xacro (robot description, xacro)
@@ -94,10 +94,14 @@
       </collision>
     </link>
-    <!-- For the Pan and Tilt joints below, velocity="1e6":
+    <!-- For the Pan and Tilt joints below, velocity="1e6" in real mode:
     URDF requires a velocity attribute on revolute joints, but hardware-enforced
     velocity profiling makes software rate-limiting redundant and causes spurious
     "command out of limits" errors from ros2_control when joy_teleop sends large absolute
     position steps. 1e6 rad/s is physically unreachable and effectively disables the
-    JointSaturationLimiter's per-cycle velocity clipping for these joints. -->
+    JointSaturationLimiter's per-cycle velocity clipping for these joints.
+    In gazebo mode there's no hardware doing that profiling - GazeboSimSystem uses this
+    same <limit velocity> to bound the simulated joint's motion, so 1e6 there would mean
+    the joint snaps to commanded position essentially instantly. Use the real computed
+    ceiling (pantilt_max_velocity_rads, pantilt.control.xacro) instead in that case. -->
     <!-- Pan joint (revolute) -->
     <joint name="pan_joint" type="revolute">
@@ -106,5 +110,5 @@
       <origin xyz="${pan_joint_x} 0 ${pan_joint_z}" rpy="0 0 0"/>
       <axis xyz="0 0 1"/>
-      <limit lower="${pan_joint_lower}" upper="${pan_joint_upper}" effort="${max_torque_nm}" velocity="1e6"/>
+      <limit lower="${pan_joint_lower}" upper="${pan_joint_upper}" effort="${max_torque_nm}" velocity="${1e6 if '$(arg ros2_control_hardware_type)' == 'real' else pantilt_max_velocity_rads}"/>
     </joint>
     <!-- Tilt joint (revolute) -->
@@ -114,5 +118,5 @@
       <origin xyz="${tilt_joint_x} 0 ${tilt_joint_z}" rpy="${tilt_joint_rx} ${tilt_joint_ry} 0"/>
       <axis xyz="0 0 -1"/>
-      <limit lower="${tilt_joint_lower}" upper="${tilt_joint_upper}" effort="${max_torque_nm}" velocity="1e6"/>
+      <limit lower="${tilt_joint_lower}" upper="${tilt_joint_upper}" effort="${max_torque_nm}" velocity="${1e6 if '$(arg ros2_control_hardware_type)' == 'real' else pantilt_max_velocity_rads}"/>
     </joint>
     <!-- OAK-D-S2 Camera + IMU -->

File: pt_description/urdf/pantilt.urdf.xacro (robot description, xacro)
@@ -17,3 +17,11 @@
 	  <origin xyz="0 0 0" rpy="0 0 0"/>
 	</xacro:pantilt_module>
+  <!-- Gazebo simulation: spawns controller_manager inside the gz_sim process, loading
+       $(arg simulation_controllers). Inert (ignored) outside Gazebo, so this is safe to
+       leave in place regardless of ros2_control_hardware_type. -->
+  <gazebo>
+    <plugin filename="gz_ros2_control-system" name="gz_ros2_control::GazeboSimROS2ControlPlugin">
+      <parameters>$(arg simulation_controllers)</parameters>
+    </plugin>
+  </gazebo>
 </robot>

Commit message: Fix pantilt torque limit and actuator damping against real STS3215 specs
max_torque_nm was documented as "30 kgf*cm for STS3215" but that figure
belongs to a different, higher-voltage (12V) member of the ST3215 family.
The actual servo used here - STS3215-C001, "matches so_arm100" per this
file's own comment - is rated 19.5 kgf*cm stall @ 7.4V per Feetech's
datasheet (cross-checked against three independent listings, including
the SO-ARM100/101 product page). Corrected to 1.9123 N*m.

That alone made overshoot worse (13% on a full-range step, up from 2%):
the real servo's firmware velocity-profiles its own trajectory and never
receives an instantaneous step, while d.ctrl here does - so the lower,
now-accurate torque ceiling saturates harder during the initial
acceleration and needs more damping margin to recover cleanly. Swept
dampratio empirically at the corrected torque and found 1.75 (up from 1)
eliminates overshoot entirely on both joints across their full range,
confirmed by stepping each to +-90 deg and checking the position trace
never exceeds the commanded target.

Also switched to MuJoCo's implicitfast integrator (their own docs call it
"a strict improvement" over the default Euler for actuator-driven models,
at equivalent cost) as general hardening, though empirically it wasn't
what was driving this particular overshoot.

No placement/geometry values touched.

Co-Authored-By: Claude Sonnet 5 <noreply@anthropic.com>

File: pt_description/urdf/pantilt.control.xacro (robot description, xacro)
@@ -41,5 +41,8 @@
        (pantilt.joints.xacro) - only used by module.xacro's gazebo-mode <limit velocity>,
        real mode keeps velocity="1e6" (see module.xacro's comment on why) regardless. -->
-  <xacro:property name="max_torque_nm"    value="2.942"/>  <!-- N⋅m (30 kgf⋅cm for STS3215) -->
+  <!-- 19.5 kgf*cm stall torque @ 7.4V per Feetech's STS3215-C001 datasheet (the SO-ARM100/101
+       variant this project uses, per pantilt_shared.xml's "matches so_arm100" comment) - not
+       the 30 kgf*cm figure, which belongs to a different 12V member of the ST3215 family. -->
+  <xacro:property name="max_torque_nm"    value="1.9123"/>  <!-- N⋅m (19.5 kgf⋅cm @ 7.4V) -->
   <xacro:property name="pantilt_max_velocity_steps" value="${int(sts_max_velocity_steps * 0.85)}"/>
   <xacro:property name="pantilt_max_velocity_rads"  value="${pantilt_max_velocity_steps * 2 * pi / 4096}"/>

File: pt_description/urdf/pt100.urdf (robot description, URDF)
Before this commit: robot pantilt, 7 links, 6 joints
Joints:
- joint pan_joint: limit lower=-1.5708 upper=1.5708 effort=2.942 velocity=1000000.0 -> lower=-1.5708 upper=1.5708 effort=1.9123 velocity=1000000.0
- joint tilt_joint: limit lower=-1.5708 upper=1.5708 effort=2.942 velocity=1000000.0 -> lower=-1.5708 upper=1.5708 effort=1.9123 velocity=1000000.0

File: pt_description/urdf/pt101.urdf (robot description, URDF)
Before this commit: robot pantilt, 7 links, 6 joints
Joints:
- joint pan_joint: limit lower=-1.5708 upper=1.5708 effort=2.942 velocity=1000000.0 -> lower=-1.5708 upper=1.5708 effort=1.9123 velocity=1000000.0
- joint tilt_joint: limit lower=-1.5708 upper=1.5708 effort=2.942 velocity=1000000.0 -> lower=-1.5708 upper=1.5708 effort=1.9123 velocity=1000000.0

Commit message: Correct STS3215 torque back to 30 kgf*cm - this project uses the 12V variant
Previous commit (5484a6c) switched to the 7.4V/19.5 kgf*cm spec, assuming
the stock SO-ARM100/101 servo - but this project actually runs the 12V
STS3215 variant, where 30 kgf*cm (2.942 N*m) is the correct stall torque.

Re-tuned dampratio empirically at the correct 2.942 N*m forcerange:
1.5 (not 1.75, which was tuned for the wrong/lower torque value) gives
0.0% overshoot on both joints across their full +-90 deg range.

Co-Authored-By: Claude Sonnet 5 <noreply@anthropic.com>

File: pt_description/urdf/pantilt.control.xacro (robot description, xacro)
@@ -41,8 +41,8 @@
        (pantilt.joints.xacro) - only used by module.xacro's gazebo-mode <limit velocity>,
        real mode keeps velocity="1e6" (see module.xacro's comment on why) regardless. -->
-  <!-- 19.5 kgf*cm stall torque @ 7.4V per Feetech's STS3215-C001 datasheet (the SO-ARM100/101
-       variant this project uses, per pantilt_shared.xml's "matches so_arm100" comment) - not
-       the 30 kgf*cm figure, which belongs to a different 12V member of the ST3215 family. -->
-  <xacro:property name="max_torque_nm"    value="1.9123"/>  <!-- N⋅m (19.5 kgf⋅cm @ 7.4V) -->
+  <!-- This project runs the 12V STS3215 variant: 30 kgf*cm stall torque per Feetech's
+       datasheet for that voltage option (not the 7.4V/19.5 kgf*cm variant used by stock
+       SO-ARM100/101). -->
+  <xacro:property name="max_torque_nm"    value="2.942"/>  <!-- N⋅m (30 kgf⋅cm @ 12V) -->
   <xacro:property name="pantilt_max_velocity_steps" value="${int(sts_max_velocity_steps * 0.85)}"/>
   <xacro:property name="pantilt_max_velocity_rads"  value="${pantilt_max_velocity_steps * 2 * pi / 4096}"/>

File: pt_description/urdf/pt100.urdf (robot description, URDF)
Before this commit: robot pantilt, 7 links, 6 joints
Joints:
- joint pan_joint: limit lower=-1.5708 upper=1.5708 effort=1.9123 velocity=1000000.0 -> lower=-1.5708 upper=1.5708 effort=2.942 velocity=1000000.0
- joint tilt_joint: limit lower=-1.5708 upper=1.5708 effort=1.9123 velocity=1000000.0 -> lower=-1.5708 upper=1.5708 effort=2.942 velocity=1000000.0

File: pt_description/urdf/pt101.urdf (robot description, URDF)
Before this commit: robot pantilt, 7 links, 6 joints
Joints:
- joint pan_joint: limit lower=-1.5708 upper=1.5708 effort=1.9123 velocity=1000000.0 -> lower=-1.5708 upper=1.5708 effort=2.942 velocity=1000000.0
- joint tilt_joint: limit lower=-1.5708 upper=1.5708 effort=1.9123 velocity=1000000.0 -> lower=-1.5708 upper=1.5708 effort=2.942 velocity=1000000.0

Commit message: Make max_velocity_steps a per-joint parameter, rename sts_max_velocity_steps
max_velocity_steps is now set on each pan/tilt joint instead of the whole
hardware bus, matching the same change in sts_hardware_interface's own
per-joint parameter support. Also renames sts_max_velocity_steps to
sts3215_max_vel_steps to make explicit that it's an STS3215-specific default,
since the underlying param is now per-motor and model-agnostic.

Co-Authored-By: Claude Sonnet 5 <noreply@anthropic.com>

File: pt_description/urdf/pantilt.control.xacro (robot description, xacro)
@@ -10,5 +10,5 @@
   <xacro:arg name="pan_center_steps"       default="2048"/>
   <xacro:arg name="tilt_center_steps"      default="2646"/>
-  <xacro:arg name="sts_max_velocity_steps" default="3400"/>   <!-- STS3215=3400, STS3032=2900, STS3235=3400 -->
+  <xacro:arg name="sts3215_max_vel_steps" default="3400"/>   <!-- STS3215=3400, STS3032=2900, STS3235=3400 -->
   <xacro:arg name="proportional_vel_max"   default="0"/>      <!-- [0-max_velocity_steps]; 0 = each joint uses commanded velocity -->
   <xacro:arg name="pan_joint_lower"        default="-1.5708"/>  <!-- rad, default -π/2 -->
@@ -32,8 +32,7 @@
   <xacro:arg name="mujoco_model" default=""/>
   <xacro:arg name="mujoco_headless" default="false"/>
-  <!-- Hardware velocity ceiling — defined before <ros2_control> because the hardware
-       plugin param references it directly. pantilt_joints receives the same value so
-       joint velocity limits stay consistent with what the interface is configured to enforce. -->
-  <xacro:property name="sts_max_velocity_steps" value="$(arg sts_max_velocity_steps)"/>
+  <!-- Motor-specific, model-dependent velocity ceiling — defined before <ros2_control>
+       because pantilt_joints (called below) writes it per joint as max_velocity_steps. -->
+  <xacro:property name="sts3215_max_vel_steps" value="$(arg sts3215_max_vel_steps)"/>
   <!-- Torque/velocity limits and joint limits as top-level properties — required by
        pantilt.module.xacro for the URDF <limit> elements on the revolute joints.
@@ -45,5 +44,5 @@
        SO-ARM100/101). -->
   <xacro:property name="max_torque_nm"    value="2.942"/>  <!-- N⋅m (30 kgf⋅cm @ 12V) -->
-  <xacro:property name="pantilt_max_velocity_steps" value="${int(sts_max_velocity_steps * 0.85)}"/>
+  <xacro:property name="pantilt_max_velocity_steps" value="${int(sts3215_max_vel_steps * 0.85)}"/>
   <xacro:property name="pantilt_max_velocity_rads"  value="${pantilt_max_velocity_steps * 2 * pi / 4096}"/>
   <xacro:property name="pan_joint_lower"  value="$(arg pan_joint_lower)"/>
@@ -70,5 +69,4 @@
         <param name="use_sync_write">$(arg use_sync_write)</param>
         <param name="enable_mock_mode">$(arg use_mock)</param>
-        <param name="max_velocity_steps">${sts_max_velocity_steps}</param>
         <param name="proportional_vel_max">$(arg proportional_vel_max)</param>
         <param name="reset_states_on_activate">true</param>
@@ -80,5 +78,5 @@
         pan_center_steps="$(arg pan_center_steps)"
         tilt_center_steps="$(arg tilt_center_steps)"
-        sts_max_velocity_steps="${sts_max_velocity_steps}"
+        sts3215_max_vel_steps="${sts3215_max_vel_steps}"
         pan_joint_lower="${pan_joint_lower}"
         pan_joint_upper="${pan_joint_upper}"

File: pt_description/urdf/pantilt.joints.xacro (robot description, xacro)
@@ -12,6 +12,6 @@
       pan_center_steps      — raw step value (0–4095) for pan centre position
       tilt_center_steps     — raw step value (0–4095) for tilt centre position
-      sts_max_velocity_steps — hardware velocity ceiling in steps/s; must match
-                               the value given to the hardware interface plugin
+      sts3215_max_vel_steps — motor's max velocity in steps/s, model-dependent;
+                               written per joint as max_velocity_steps
   -->
   <xacro:macro name="pantilt_joints" params="
@@ -20,5 +20,5 @@
       pan_center_steps:=2048
       tilt_center_steps:=2646
-      sts_max_velocity_steps:=3400
+      sts3215_max_vel_steps:=3400
       pan_joint_lower:=-1.5708
       pan_joint_upper:=1.5708
@@ -27,5 +27,5 @@
       ros2_control_hardware_type:=real">
     <!-- 85% of hardware max — 15% safety margin; motor firmware handles profiling -->
-    <xacro:property name="pantilt_max_velocity_steps" value="${int(sts_max_velocity_steps * 0.85)}"/>
+    <xacro:property name="pantilt_max_velocity_steps" value="${int(sts3215_max_vel_steps * 0.85)}"/>
     <xacro:property name="pantilt_max_velocity_rads"  value="${pantilt_max_velocity_steps * 2 * pi / 4096}"/>
     <!-- Pan axis: rotates the payload around Z -->
@@ -35,4 +35,6 @@
       <param name="min_position">${pan_joint_lower}</param>
       <param name="max_position">${pan_joint_upper}</param>
+      <!-- Motor-specific, model-dependent parameter (per joint so different STS models can share this bus) -->
+      <param name="max_velocity_steps">${sts3215_max_vel_steps}</param>
       <param name="max_velocity">${pantilt_max_velocity_rads}</param>
       <param name="position_center_steps">${pan_center_steps}</param>
@@ -57,4 +59,6 @@
       <param name="min_position">${tilt_joint_lower}</param>
       <param name="max_position">${tilt_joint_upper}</param>
+      <!-- Motor-specific, model-dependent parameter (per joint so different STS models can share this bus) -->
+      <param name="max_velocity_steps">${sts3215_max_vel_steps}</param>
       <param name="max_velocity">${pantilt_max_velocity_rads}</param>
       <param name="position_center_steps">${tilt_center_steps}</param>
