Commit message: Trim verbose comments/docs, fix stale artifacts
Comments in the MuJoCo/xacro files and README had grown into
multi-paragraph narratives (debugging journeys, alternatives
considered, specific validation numbers) rather than the facts
needed to safely modify the code. Trimmed throughout, and cut the
README's Design/Simulation sections down since simulation is a
minor, lightly-tested part of this package.

Also fixes real issues found along the way:
- pt100.urdf/pt101.urdf were stale, missing the <gazebo> plugin
  block and other content added since they were last regenerated -
  regenerated both.
- oakd_s2.module.xacro's macro comment said "for pt100 only" -
  wrong, it's shared by both variants.
- pt_bringup's CMake target was named colored_pointcloud_compressor_node,
  matching no other identifier in the package (source file/class/
  executable are all pcl_compressor_node/PCLCompressorNode/
  pcl_compressor) - renamed for consistency.

Co-Authored-By: Claude Sonnet 5 <noreply@anthropic.com>

File: pt_description/mjcf/pantilt.mjcf.xacro (robot description, xacro)
@@ -1,57 +1,25 @@
 <?xml version="1.0"?>
-<!-- Parametric PT100/PT101 MJCF assembly - the mujoco_ros2_control equivalent of
-     pantilt.module.xacro *and* pantilt.urdf.xacro combined: defines the pantilt_body macro
-     plus the mesh/property selection it depends on (driven by the SAME pantilt_config arg
-     used throughout the URDF side - pantilt.common.xacro:pantilt_config - rather than a
-     separate near-duplicate file per variant), and - only when used standalone, see
-     `standalone` below - invokes that macro directly in worldbody plus a floor/lighting
-     scene for direct viewing.
-     Standalone use (`standalone` defaults to true):
-       xacro pantilt.mjcf.xacro pantilt_config:=pt101 > /tmp/pantilt.xml
-       python3 -m mujoco.viewer, mjcf flag pointed at /tmp/pantilt.xml
-     pt_control/launch/pantilt.launch.py runs this same command at launch time (sim:=true)
-     and writes the result to a temp file, passed as mujoco_model.
-     Embedded use (lekiwi_ros2's base_pantilt.mjcf.xacro, base + payload combined): included
-     via xacro:include with the `pantilt_body` macro invoked at whatever mount point the
-     includer chooses, and the worldbody+scene block below suppressed - the includer declares
-     its OWN `<xacro:arg name="standalone" default="false"/>` *before* including this file,
-     which wins over this file's own `default="true"` (xacro resolves an arg's default from
-     whichever `<xacro:arg>` declaration is encountered FIRST in processing order, confirmed
-     empirically - a later re-declaration of the same arg name is silently ignored, so the
-     includer declaring it first is what makes this safe without also having to remember to
-     pass `standalone:=false` explicitly on every xacro invocation). Without this, embedding
-     would duplicate the whole pan-tilt assembly - a stray top-level worldbody with a second
-     pantilt_base_link, in addition to the correctly-mounted one (hit this for real before
-     splitting worldbody-emission out behind this arg).
-     Processed with the `xacro` CLI, same tool and convention as every other file in this
-     project's urdf/ trees - MJCF has no native macro/conditional system of its own, so this
-     reuses xacro instead of hand-duplicating pt100_oakd_s2.xml/pt101_oakd_s2.xml (the
-     two-static-file approach used in this file's own first draft, replaced here).
-     $(find pt_description) is used for every cross-file reference instead of a relative
-     path, so this resolves correctly regardless of where the FINAL xacro-processed output
-     ends up (a launch-time temp file, not necessarily this file's own directory) - unlike
-     raw MJCF's own <include>, which only supports filesystem-relative paths with no
-     $(find)-equivalent. -->
+<!-- Parametric PT100/PT101 MJCF assembly (mujoco_ros2_control equivalent of
+     pantilt.module.xacro + pantilt.urdf.xacro): defines the pantilt_body macro, selected by
+     pantilt_config, and when standalone:=true (default) invokes it in worldbody plus a
+     floor/lighting scene.
+     Standalone: xacro pantilt.mjcf.xacro pantilt_config:=pt101 > /tmp/pantilt.xml
+     pt_control/launch/pantilt.launch.py runs the same command at launch time.
+     Embedded (lekiwi_ros2's base_pantilt.mjcf.xacro): the includer declares its own
+     standalone:=false BEFORE including this file, which wins - xacro takes the first
+     <xacro:arg> declaration of a given name, later ones are ignored - and invokes
+     pantilt_body itself at its own mount point. Without this the worldbody+scene block
+     below would duplicate the whole assembly. -->
 <mujoco xmlns:xacro="http://www.ros.org/wiki/xacro" model="pantilt">
   <xacro:arg name="pantilt_config" default="pt101"/>
   <xacro:arg name="standalone" default="true"/>
   <xacro:property name="pantilt_config" value="$(arg pantilt_config)"/>
-  <!-- xacro:include (a full text-level splice at xacro-PROCESS time), not a plain MJCF
-       <include> - pantilt_shared.xml's own mesh file= paths use $(find pt_description),
-       which only xacro itself resolves; a plain <include> would leave that text
-       unprocessed for MuJoCo to choke on. See pantilt_shared.xml's own header comment for
-       why its meshdir was replaced with absolute paths in the first place. -->
+  <!-- xacro:include, not a plain <include> - pantilt_shared.xml's mesh paths use $(find),
+       which only xacro resolves. -->
   <xacro:include filename="$(find pt_description)/mjcf/pantilt_shared.xml"/>
   <!-- Mesh files and mesh-local offset corrections - pt100 defaults below, overridden for
-       pt101. Values match pt_description/urdf/pantilt.common.xacro's own
-       pantilt_base_mesh/pan_joint_mesh/*_rpy/*_xyz properties in spirit (same physical
-       corrections), but are NOT literally $(find)-included from that file and reused
-       as-is: URDF's rpy and MuJoCo's default euler attribute do not compose rotations in
-       the same order (confirmed empirically - lekiwi_ros2's base_shared.xml has the same
-       caveat in its own wheel-orientation comment), so porting a multi-axis rpy value
-       directly as a MuJoCo euler value is only safe to verify case-by-case, not to assume. These
-       euler values are ported from and identical to what shipped in this project's
-       original (pre-parametrization) pt100_oakd_s2.xml/pt101_oakd_s2.xml files, each
-       validated individually before this file merged them - not re-derived here. -->
+       pt101. Not $(find)-included from pantilt.common.xacro's equivalent properties: URDF's
+       rpy and MuJoCo's euler don't compose rotations the same way, so these were each
+       independently validated rather than ported directly. -->
   <xacro:property name="pantilt_base_mesh" value="pantilt_base_100.stl"/>
   <xacro:property name="pan_link_mesh_file" value="pan_joint_100.stl"/>
@@ -72,9 +40,7 @@
     <mesh name="pan_link_mesh" file="$(find pt_description)/meshes/${pan_link_mesh_file}"/>
   </asset>
-  <!-- pantilt_base_link carries no pos/euler of its own - it inherits whichever frame the
-       invocation site provides (worldbody below for standalone use, or a mount body in
-       lekiwi_ros2's base_pantilt.mjcf.xacro for the combined base+payload case). Collision
-       geoms match pantilt.module.xacro exactly: only the primary body mesh, not the
-       decorative "_motor" sub-meshes. -->
+  <!-- pantilt_base_link has no pos/euler of its own - it inherits the invocation site's
+       frame. Collision geoms cover only the primary body mesh, not the decorative "_motor"
+       sub-meshes. -->
   <xacro:macro name="pantilt_body">
     <body name="pantilt_base_link">
@@ -100,8 +66,7 @@
     </body>
   </xacro:macro>
-  <!-- Compares $(arg standalone) directly rather than through a bridged <xacro:property> -
-       xacro auto-coerces a property whose value is the literal string "true"/"false" into a
-       Python bool, so ${standalone == 'true'} would silently compare True (bool) == 'true'
-       (str) and always be False (confirmed empirically). -->
+  <!-- Compares $(arg standalone) directly, not via a bridged <xacro:property> - xacro
+       auto-coerces "true"/"false" property values to Python bool, breaking a naive
+       string comparison. -->
   <xacro:if value="${'$(arg standalone)' == 'true'}">
     <worldbody>

File: pt_description/urdf/oakd_s2.module.xacro (robot description, xacro)
@@ -3,5 +3,5 @@
 	xmlns:xacro="http://ros.org/wiki/xacro">
 	<!--
-	  Custom OAK-D-S2 camera macro for pt100 only.
+	  Custom OAK-D-S2 camera macro, shared by both pt100/pt101.
 	  This version allows direct color parameterization (r/g/b/a) for the mesh material.
 	-->

File: pt_description/urdf/pantilt.module.xacro (robot description, xacro)
@@ -94,14 +94,8 @@
       </collision>
     </link>
-    <!-- For the Pan and Tilt joints below, velocity="1e6" in real mode:
-    URDF requires a velocity attribute on revolute joints, but hardware-enforced
-    velocity profiling makes software rate-limiting redundant and causes spurious
-    "command out of limits" errors from ros2_control when joy_teleop sends large absolute
-    position steps. 1e6 rad/s is physically unreachable and effectively disables the
-    JointSaturationLimiter's per-cycle velocity clipping for these joints.
-    In gazebo mode there's no hardware doing that profiling - GazeboSimSystem uses this
-    same <limit velocity> to bound the simulated joint's motion, so 1e6 there would mean
-    the joint snaps to commanded position essentially instantly. Use the real computed
-    ceiling (pantilt_max_velocity_rads, pantilt.control.xacro) instead in that case. -->
+    <!-- real mode: velocity="1e6" (unreachable) disables JointSaturationLimiter's clipping,
+         since joy_teleop's absolute position jumps would otherwise trip spurious limit
+         errors. gazebo mode: uses the real computed ceiling instead, since GazeboSimSystem
+         actually enforces this limit on the simulated joint. -->
     <!-- Pan joint (revolute) -->
     <joint name="pan_joint" type="revolute">

File: pt_description/urdf/pt100.urdf (robot description, URDF)
Before this commit: robot pantilt, 7 links, 6 joints
Joints:
- joint pan_joint: limit lower=-1.5708 upper=1.5708 effort=2.942 velocity=1e6 -> lower=-1.5708 upper=1.5708 effort=2.942 velocity=1000000.0
- joint tilt_joint: limit lower=-1.5708 upper=1.5708 effort=2.942 velocity=1e6 -> lower=-1.5708 upper=1.5708 effort=2.942 velocity=1000000.0

File: pt_description/urdf/pt101.urdf (robot description, URDF)
Before this commit: robot pantilt, 7 links, 6 joints
Joints:
- joint pan_joint: limit lower=-1.5708 upper=1.5708 effort=2.942 velocity=1e6 -> lower=-1.5708 upper=1.5708 effort=2.942 velocity=1000000.0
- joint tilt_joint: limit lower=-1.5708 upper=1.5708 effort=2.942 velocity=1e6 -> lower=-1.5708 upper=1.5708 effort=2.942 velocity=1000000.0

Commit message: Fix pantilt mesh placement: MuJoCo euler order differs from URDF rpy
URDF's rpy composes as Rz*Ry*Rx (fixed-axis roll,pitch,yaw); MuJoCo's
default euler="xyz" composes as Rx*Ry*Rz - the reverse order. These only
agree when rpy has a single nonzero axis. Every multi-axis rotation in the
pantilt assembly (pantilt_base_link mesh, pan_link mesh, tilt_motor,
tilt_link body, tilt_joint_oakd_s2 mesh, oak_link body, oak_link_model_origin
body) was ported directly from URDF rpy values into MJCF euler, scattering
the OAK-D camera and pan/tilt meshes across the scene instead of assembling
them. Replaced each with a quat computed directly from the URDF's own rpy
convention. Verified by comparing every body's world pose against a
from-scratch URDF forward-kinematics computation (pt100 and pt101) - all
now match exactly, where they previously diverged by centimeters.

Co-Authored-By: Claude Sonnet 5 <noreply@anthropic.com>

File: pt_description/mjcf/pantilt.mjcf.xacro (robot description, xacro)
@@ -20,19 +20,21 @@
   <!-- Mesh files and mesh-local offset corrections - pt100 defaults below, overridden for
        pt101. Not $(find)-included from pantilt.common.xacro's equivalent properties: URDF's
-       rpy and MuJoCo's euler don't compose rotations the same way, so these were each
-       independently validated rather than ported directly. -->
+       rpy composes as Rz*Ry*Rx (fixed-axis roll,pitch,yaw) while MuJoCo's default euler="xyz"
+       composes as Rx*Ry*Rz - the reverse order. These only agree when rpy has a single nonzero
+       axis; every offset below has 2+ nonzero axes, so each is given as a quat computed
+       directly from the URDF's rpy (via its own Rz*Ry*Rx convention), not a ported euler. -->
   <xacro:property name="pantilt_base_mesh" value="pantilt_base_100.stl"/>
   <xacro:property name="pan_link_mesh_file" value="pan_joint_100.stl"/>
   <xacro:property name="pantilt_base_geom_pos" value="0 0 0"/>
-  <xacro:property name="pantilt_base_geom_euler" value="0 0 1.5707963267948966"/>
+  <xacro:property name="pantilt_base_geom_quat" value="0.5 0.5 0.5 0.5"/>
   <xacro:property name="pan_link_geom_pos" value="0 0 0"/>
-  <xacro:property name="pan_link_geom_euler" value="1.5707963267948966 0 1.5707963267948966"/>
+  <xacro:property name="pan_link_geom_quat" value="0.5 0.5 0.5 0.5"/>
   <xacro:if value="${pantilt_config == 'pt101'}">
     <xacro:property name="pantilt_base_mesh" value="pantilt_base_101.stl"/>
     <xacro:property name="pan_link_mesh_file" value="pan_joint_101.stl"/>
     <xacro:property name="pantilt_base_geom_pos" value="0 0 0.0002"/>
-    <xacro:property name="pantilt_base_geom_euler" value="1.5707963267948966 0 1.5707963267948966"/>
+    <xacro:property name="pantilt_base_geom_quat" value="0.5 0.5 0.5 0.5"/>
     <xacro:property name="pan_link_geom_pos" value="-0.0120 0 0.00205"/>
-    <xacro:property name="pan_link_geom_euler" value="1.5707963267948966 0 3.141592653589793"/>
+    <xacro:property name="pan_link_geom_quat" value="0.0 0.0 0.70710678 0.70710678"/>
   </xacro:if>
   <asset>
@@ -47,9 +49,9 @@
       <inertial pos="0 0 0" mass="1.0" diaginertia="0.01 0.01 0.01"/>
       <geom mesh="pantilt_base_link_mesh" material="light_grey" class="visual"
-            pos="${pantilt_base_geom_pos}" euler="${pantilt_base_geom_euler}"/>
+            pos="${pantilt_base_geom_pos}" quat="${pantilt_base_geom_quat}"/>
       <geom mesh="pan_motor" material="charcoal" class="visual"
             pos="0 0 0" euler="0 0 1.5707963267948966"/>
       <geom mesh="pantilt_base_link_mesh" class="collision"
-            pos="${pantilt_base_geom_pos}" euler="${pantilt_base_geom_euler}"/>
+            pos="${pantilt_base_geom_pos}" quat="${pantilt_base_geom_quat}"/>
       <body name="pan_link" pos="0.0452 0 0.0165">
         <inertial pos="-9.07886e-05 0.0590972 0.031089" mass="0.119226"
@@ -57,9 +59,9 @@
         <joint name="pan_joint" class="pan"/>
         <geom mesh="pan_link_mesh" material="light_grey" class="visual"
-              pos="${pan_link_geom_pos}" euler="${pan_link_geom_euler}"/>
+              pos="${pan_link_geom_pos}" quat="${pan_link_geom_quat}"/>
         <geom mesh="tilt_motor" material="charcoal" class="visual"
-              pos="0 0 0" euler="1.5707963267948966 0 1.5707963267948966"/>
+              pos="0 0 0" quat="0.5 0.5 0.5 0.5"/>
         <geom mesh="pan_link_mesh" class="collision"
-              pos="${pan_link_geom_pos}" euler="${pan_link_geom_euler}"/>
+              pos="${pan_link_geom_pos}" quat="${pan_link_geom_quat}"/>
         <include file="$(find pt_description)/mjcf/oakd_s2_subtree.xml"/>
       </body>

Commit message: Fix pantilt_base_link_mesh orientation for pt100 - wrong quat, not pt101's
pantilt_base_geom_quat's pt100 default was "0.5 0.5 0.5 0.5" - the value
correctly computed for pt101's pantilt_base_101.stl (URDF rpy = pi/2, 0,
pi/2), copy-pasted into the pt100 default slot instead of computing
pt100's own value. pantilt_base_100.stl's actual URDF origin is rpy =
0, 0, pi/2 (single Z axis only), so it needs Rz(90) alone, not the same
quat as pt101's two-axis rotation.

Caught because pt101 was correct and pt100 wasn't, despite both going
through the same fix in 89eb0b9 - narrowed down by re-verifying every
mesh geom's quat against a fresh point-cloud (not just bounding-box)
comparison to the URDF-rotated raw STL: pantilt_base_100.stl was off by
9mm mean / 25.5mm max with the old quat, exact 0.000mm with the fix.
pan_joint_100.stl (the other pt100-specific mesh) was already correct.

Co-Authored-By: Claude Sonnet 5 <noreply@anthropic.com>

File: pt_description/mjcf/pantilt.mjcf.xacro (robot description, xacro)
@@ -27,5 +27,7 @@
   <xacro:property name="pan_link_mesh_file" value="pan_joint_100.stl"/>
   <xacro:property name="pantilt_base_geom_pos" value="0 0 0"/>
-  <xacro:property name="pantilt_base_geom_quat" value="0.5 0.5 0.5 0.5"/>
+  <!-- pt100's pantilt_base_100.stl URDF origin is rpy="0 0 pi/2" (single Z axis, unlike
+       pt101's) - quat is Rz(90) alone, not pt101's override value below. -->
+  <xacro:property name="pantilt_base_geom_quat" value="0.70710678 0 0 0.70710678"/>
   <xacro:property name="pan_link_geom_pos" value="0 0 0"/>
   <xacro:property name="pan_link_geom_quat" value="0.5 0.5 0.5 0.5"/>
