Commit message: Align pt101/pt100 with so101/so100 conventions, add tests, single-source-of-truth config
Brings pantilt_ros2 closer to structural parity with so_arm_ros2 (treated as the
reference implementation for a repurposed SO-ARM100/101 first-two-joints device):

- Fix pan_joint's origin-to-mesh alignment: pan_link's own-link mesh bbox now sits
  relative to pan_joint's origin the same way SO101's shoulder_link sits relative to
  shoulder_pan_joint (verified via STL bounding-box measurement against so101.urdf).
  Zero world-space regression - pan_joint's axis was resliced with an equal-and-opposite
  compensation on pan_link's own mesh content, verified via mesh-vertex-world-position
  diff (max 2.8e-17m) and FK diff on tilt_joint/tilt_link/oak_link/oak_imu_frame (zero
  diff at rest and at arbitrary joint angles). pt100 needed no change - confirmed exact
  match (delta=0.0) to SO100's own convention already.

- Rename pan_joint/pan_link -> shoulder_pan_joint/shoulder_link (and matching internal
  xacro properties) to match so101/so100's own joint/link naming, across pt_description's
  URDF/xacro and MJCF files.

- Motor IDs, step-centering, and joint limits are no longer duplicated in
  pt_control/config/urdf_config.yaml - they're now baked into pantilt.joints.xacro's
  macro defaults as the single source of truth, matching so101.control.xacro/
  so100.control.xacro's convention. Also fixes a latent bug: the macro's own
  tilt_center_steps default was stale at 2646 (real value 2048), never visible since
  urdf_config.yaml always overrode it.

- controller-manager spawner naming: -c /controller_manager -> -c controller_manager,
  matching so_arm_control's relative naming.

- Add pt_description/test/test_urdf_xacro.py, modeled on so_arm_description's own -
  xacro-processing + XML-structure smoke tests (joint limits, ros2_control coverage,
  mesh existence, hardware-plugin selection, parent-child chain, MJCF processing).
  pt_description had no test suite before this.

- Add detect-private-key, check-added-large-files, and actionlint pre-commit hooks,
  matching so_arm_ros2's .pre-commit-config.yaml.

Regenerated pt101.urdf/pt100.urdf and the pt100/pt101_oakd_s2.xml MJCF snapshots to
match. lekiwi_ros2's own base_pantilt.* files and control.launch.py/urdf_config.yaml
updated to match in a companion commit there.

Co-Authored-By: Claude Sonnet 5 <noreply@anthropic.com>

File: pt_description/mjcf/pantilt.mjcf.xacro (robot description, xacro)
@@ -25,22 +25,26 @@
        directly from the URDF's rpy (via its own Rz*Ry*Rx convention), not a ported euler. -->
   <xacro:property name="pantilt_base_mesh" value="pantilt_base_100.stl"/>
-  <xacro:property name="pan_link_mesh_file" value="pan_joint_100.stl"/>
+  <xacro:property name="shoulder_link_mesh_file" value="pan_joint_100.stl"/>
   <xacro:property name="pantilt_base_geom_pos" value="0 0 0"/>
   <!-- pt100's pantilt_base_100.stl URDF origin is rpy="0 0 pi/2" (single Z axis, unlike
        pt101's) - quat is Rz(90) alone, not pt101's override value below. -->
   <xacro:property name="pantilt_base_geom_quat" value="0.70710678 0 0 0.70710678"/>
-  <xacro:property name="pan_link_geom_pos" value="0 0 0"/>
-  <xacro:property name="pan_link_geom_quat" value="0.5 0.5 0.5 0.5"/>
+  <!-- shoulder_link_geom_pos Z carries the same -0.0483559 reslice compensation as
+       pantilt.common.xacro's shoulder_pan_mesh_xyz (URDF side) - see that file's comment
+       for the derivation. Applies to both configs; only X differs (pt101's bracket mesh
+       has a nonzero local X offset, pt100's doesn't). -->
+  <xacro:property name="shoulder_link_geom_pos" value="0 0 -0.0483559"/>
+  <xacro:property name="shoulder_link_geom_quat" value="0.5 0.5 0.5 0.5"/>
   <xacro:if value="${pantilt_config == 'pt101'}">
     <xacro:property name="pantilt_base_mesh" value="pantilt_base_101.stl"/>
-    <xacro:property name="pan_link_mesh_file" value="pan_joint_101.stl"/>
+    <xacro:property name="shoulder_link_mesh_file" value="pan_joint_101.stl"/>
     <xacro:property name="pantilt_base_geom_pos" value="0 0 0.0002"/>
     <xacro:property name="pantilt_base_geom_quat" value="0.5 0.5 0.5 0.5"/>
-    <xacro:property name="pan_link_geom_pos" value="-0.0120 0 0.00205"/>
-    <xacro:property name="pan_link_geom_quat" value="0.0 0.0 0.70710678 0.70710678"/>
+    <xacro:property name="shoulder_link_geom_pos" value="-0.0120 0 -0.0463059"/>
+    <xacro:property name="shoulder_link_geom_quat" value="0.0 0.0 0.70710678 0.70710678"/>
   </xacro:if>
   <asset>
     <mesh name="pantilt_base_link_mesh" file="$(find pt_description)/meshes/${pantilt_base_mesh}"/>
-    <mesh name="pan_link_mesh" file="$(find pt_description)/meshes/${pan_link_mesh_file}"/>
+    <mesh name="shoulder_link_mesh" file="$(find pt_description)/meshes/${shoulder_link_mesh_file}"/>
   </asset>
   <!-- pantilt_base_link has no pos/euler of its own - it inherits the invocation site's
@@ -60,14 +64,17 @@
       <geom mesh="pantilt_base_link_mesh" class="collision"
             pos="${pantilt_base_geom_pos}" quat="${pantilt_base_geom_quat}"/>
-      <body name="pan_link" pos="0.0452 0 0.0165">
-        <inertial pos="-9.07886e-05 0.0590972 0.031089" mass="0.119226"
+      <!-- pos Z = 0.0648559 (was 0.0165): same reslice as pantilt.common.xacro's
+           shoulder_pan_z (URDF side) - the joint origin moved along its own rotation axis,
+           compensated by the mesh offsets above/below so nothing renders differently. -->
+      <body name="shoulder_link" pos="0.0452 0 0.0648559">
+        <inertial pos="-9.07886e-05 0.0590972 -0.0172669" mass="0.119226"
                   diaginertia="5.94278e-05 5.89975e-05 3.13712e-05"/>
-        <joint name="pan_joint" class="pan"/>
-        <geom mesh="pan_link_mesh" material="light_grey" class="visual"
-              pos="${pan_link_geom_pos}" quat="${pan_link_geom_quat}"/>
+        <joint name="shoulder_pan_joint" class="pan"/>
+        <geom mesh="shoulder_link_mesh" material="light_grey" class="visual"
+              pos="${shoulder_link_geom_pos}" quat="${shoulder_link_geom_quat}"/>
         <geom mesh="tilt_motor" material="charcoal" class="visual"
-              pos="0 0 0" quat="0.5 0.5 0.5 0.5"/>
-        <geom mesh="pan_link_mesh" class="collision"
-              pos="${pan_link_geom_pos}" quat="${pan_link_geom_quat}"/>
+              pos="0 0 -0.0483559" quat="0.5 0.5 0.5 0.5"/>
+        <geom mesh="shoulder_link_mesh" class="collision"
+              pos="${shoulder_link_geom_pos}" quat="${shoulder_link_geom_quat}"/>
         <include file="$(find pt_description)/mjcf/oakd_s2_subtree.xml"/>
       </body>

File: pt_description/urdf/pantilt.common.xacro (robot description, xacro)
@@ -5,5 +5,5 @@
   <xacro:property name="charcoal_rgba" value="0.15 0.15 0.15 1.0"/>
   <xacro:property name="charcoal_rgb" value="0.15"/>
-  <!-- Pan-tilt mechanical configuration: selects pantilt_base / pan_joint mesh
+  <!-- Pan-tilt mechanical configuration: selects pantilt_base / shoulder_pan mesh
        variants. "pt101" (default, recommended) uses the SO-ARM101-based
        meshes; "pt100" uses the original SO-ARM100-based meshes. All
@@ -15,12 +15,12 @@
   <!-- Pantilt base visual compensation / mount rotation (rad) -->
   <xacro:property name="pantilt_offset_rz" value="${pi/2}"/>
-  <!-- Pan link visual compensation (rad) -->
-  <xacro:property name="pan_offset_rx" value="${pi/2}"/>
-  <xacro:property name="pan_offset_rz" value="${pi/2}"/>
+  <!-- Shoulder link visual compensation (rad) -->
+  <xacro:property name="shoulder_offset_rx" value="${pi/2}"/>
+  <xacro:property name="shoulder_offset_rz" value="${pi/2}"/>
   <xacro:property name="pantilt_base_mesh" value="pantilt_base_100.stl"/>
-  <xacro:property name="pan_joint_mesh" value="pan_joint_100.stl"/>
+  <xacro:property name="shoulder_pan_mesh" value="pan_joint_100.stl"/>
   <!-- Mesh-local origin correction, applied to the body mesh of each link
        only (not the motor meshes), in place of the shared
-       pantilt_offset_rz / pan_offset_rx+rz rotations above. pt100 meshes
+       pantilt_offset_rz / shoulder_offset_rx+rz rotations above. pt100 meshes
        reuse those shared rotations with zero translation (no-op). pt101
        meshes need a different rotation (SO-ARM101's base_link/shoulder_link
@@ -28,21 +28,37 @@
        translation; see derivation below. -->
   <xacro:property name="pantilt_base_mesh_rpy" value="0 0 ${pantilt_offset_rz}"/>
-  <xacro:property name="pan_joint_mesh_rpy" value="${pan_offset_rx} 0 ${pan_offset_rz}"/>
+  <xacro:property name="shoulder_pan_mesh_rpy" value="${shoulder_offset_rx} 0 ${shoulder_offset_rz}"/>
   <xacro:property name="pantilt_base_mesh_xyz" value="0 0 0"/>
-  <xacro:property name="pan_joint_mesh_xyz" value="0 0 0"/>
+  <xacro:property name="shoulder_pan_mesh_xyz" value="0 0 -0.0483559"/>
   <xacro:if value="${pantilt_config == 'pt101'}">
     <xacro:property name="pantilt_base_mesh" value="pantilt_base_101.stl"/>
-    <xacro:property name="pan_joint_mesh" value="pan_joint_101.stl"/>
+    <xacro:property name="shoulder_pan_mesh" value="pan_joint_101.stl"/>
     <xacro:property name="pantilt_base_mesh_rpy" value="${pi/2} 0 ${pi/2}"/>
-    <xacro:property name="pan_joint_mesh_rpy" value="${pi/2} 0 ${pi}"/>
+    <xacro:property name="shoulder_pan_mesh_rpy" value="${pi/2} 0 ${pi}"/>
     <xacro:property name="pantilt_base_mesh_xyz" value="0 0 0.0002"/>
-    <xacro:property name="pan_joint_mesh_xyz" value="-0.0120 0 0.00205"/>
+    <xacro:property name="shoulder_pan_mesh_xyz" value="-0.0120 0 -0.0463059"/>
   </xacro:if>
-  <!-- Pan joint origin (in reoriented base_link frame) -->
-  <xacro:property name="pan_joint_x" value="0.0452"/>
-  <xacro:property name="pan_joint_z" value="0.0165"/>
-  <!-- Tilt joint origin (in pan_link frame — same as SO100 shoulder_lift) -->
+  <!-- Shoulder-pan joint origin (in reoriented base_link frame). Z is offset +0.0483559 from
+       the raw SO100-derived value (0.0165) so shoulder_pan_joint's origin sits relative to
+       shoulder_link's own mesh the same way SO101's shoulder_pan_joint sits relative to
+       shoulder_link (mesh-bbox-vs-origin alignment verified against so101.urdf);
+       shoulder_pan_mesh_xyz and tilt_motor's mesh offset above/below carry the
+       equal-and-opposite compensation so no visual or downstream frame (tilt_joint,
+       tilt_link, oak_link) moves. -->
+  <xacro:property name="shoulder_pan_x" value="0.0452"/>
+  <xacro:property name="shoulder_pan_z" value="0.0648559"/>
+  <!-- Joint limits - single source of truth for pantilt.module.xacro's URDF <limit> elements
+       (needed as globals here, not macro params, since pantilt.module.xacro always includes
+       this file directly - see pantilt.joints.xacro's own matching defaults, used separately
+       for its ros2_control <joint> blocks). -->
+  <xacro:property name="shoulder_pan_lower" value="-1.5708"/>
+  <xacro:property name="shoulder_pan_upper" value="1.5708"/>
+  <xacro:property name="tilt_joint_lower" value="-1.5708"/>
+  <xacro:property name="tilt_joint_upper" value="1.5708"/>
+  <!-- Tilt joint origin (in shoulder_link frame — same as SO100 shoulder_lift, minus the same
+       -0.0483559 compensation applied to shoulder_pan_z above, so shoulder_pan_z + tilt_joint_z
+       — and therefore tilt_link's world pose — is unchanged). -->
   <xacro:property name="tilt_joint_x" value="0.0306"/>
-  <xacro:property name="tilt_joint_z" value="0.1025"/>
+  <xacro:property name="tilt_joint_z" value="0.0541441"/>
   <!-- Tilt joint frame rotation (makes Z the tilt axis, +θ = forward) -->
   <xacro:property name="tilt_joint_rx" value="${-pi/2}"/>
@@ -51,6 +67,6 @@
   <xacro:property name="tilt_offset_rx" value="${pi/2}"/>
   <xacro:property name="tilt_offset_ry" value="${-pi/2}"/>
-  <xacro:property name="tilt_visual_x" value="${pan_joint_z + tilt_joint_z}"/>
-  <xacro:property name="tilt_visual_y" value="${pan_joint_x + tilt_joint_x}"/>
+  <xacro:property name="tilt_visual_x" value="${shoulder_pan_z + tilt_joint_z}"/>
+  <xacro:property name="tilt_visual_y" value="${shoulder_pan_x + tilt_joint_x}"/>
   <xacro:property name="tilt_visual_z" value="-0.0002"/>
   <!-- OAK-D-S2 camera mount offset (in tilt_link frame) -->

File: pt_description/urdf/pantilt.control.xacro (robot description, xacro)
@@ -6,14 +6,15 @@
   <xacro:arg name="use_mock"               default="false"/>
   <xacro:arg name="use_sync_write"         default="true"/>
-  <xacro:arg name="pan_motor_id"           default="1"/>
-  <xacro:arg name="tilt_motor_id"          default="2"/>
-  <xacro:arg name="pan_center_steps"       default="2048"/>
-  <xacro:arg name="tilt_center_steps"      default="2646"/>
   <xacro:arg name="sts3215_max_vel_steps" default="3400"/>   <!-- STS3215=3400, STS3032=2900, STS3235=3400 -->
   <xacro:arg name="proportional_vel_max"   default="0"/>      <!-- [0-max_velocity_steps]; 0 = each joint uses commanded velocity -->
-  <xacro:arg name="pan_joint_lower"        default="-1.5708"/>  <!-- rad, default -π/2 -->
-  <xacro:arg name="pan_joint_upper"        default="1.5708"/>   <!-- rad, default +π/2 -->
-  <xacro:arg name="tilt_joint_lower"       default="-1.5708"/>  <!-- rad, default -π/2 -->
-  <xacro:arg name="tilt_joint_upper"       default="1.5708"/>   <!-- rad, default +π/2 -->
+  <!-- Motor IDs, step-centering, and joint limits are NOT xacro:args here - they're
+       physical-calibration constants for this mechanism (motor wiring, servo centering),
+       not per-deployment connection settings, so pantilt.joints.xacro's macro defaults are
+       their single source of truth (same convention as so101.control.xacro/so100.control.xacro
+       in so_arm_ros2, which hardcode motor IDs/joint limits as fixed xacro:property values
+       rather than sourcing them from an external launch-time YAML). A host embedding this
+       mechanism on a shared bus (e.g. lekiwi_ros2's base_pantilt.control.xacro) can still
+       override any of pantilt_joints' macro params explicitly if it ever needs different
+       values - see pantilt.joints.xacro. -->
   <!-- Simulation -->
   <!-- "real" (default) keeps the STS3215 serial hardware plugin below unchanged.
@@ -35,6 +36,6 @@
        because pantilt_joints (called below) writes it per joint as max_velocity_steps. -->
   <xacro:property name="sts3215_max_vel_steps" value="$(arg sts3215_max_vel_steps)"/>
-  <!-- Torque/velocity limits and joint limits as top-level properties — required by
-       pantilt.module.xacro for the URDF <limit> elements on the revolute joints.
+  <!-- Torque limit as a top-level property — required by pantilt.module.xacro for the URDF
+       <limit> elements on the revolute joints.
        pantilt_max_velocity_rads duplicates pantilt_joints' own local computation
        (pantilt.joints.xacro) - only used by module.xacro's gazebo-mode <limit velocity>,
@@ -46,8 +47,4 @@
   <xacro:property name="pantilt_max_velocity_steps" value="${int(sts3215_max_vel_steps * 0.85)}"/>
   <xacro:property name="pantilt_max_velocity_rads"  value="${pantilt_max_velocity_steps * 2 * pi / 4096}"/>
-  <xacro:property name="pan_joint_lower"  value="$(arg pan_joint_lower)"/>
-  <xacro:property name="pan_joint_upper"  value="$(arg pan_joint_upper)"/>
-  <xacro:property name="tilt_joint_lower" value="$(arg tilt_joint_lower)"/>
-  <xacro:property name="tilt_joint_upper" value="$(arg tilt_joint_upper)"/>
   <xacro:include filename="$(find pt_description)/urdf/pantilt.joints.xacro"/>
   <!-- ROS 2 CONTROL -->
@@ -74,13 +71,5 @@
     </hardware>
     <xacro:pantilt_joints
-        pan_motor_id="$(arg pan_motor_id)"
-        tilt_motor_id="$(arg tilt_motor_id)"
-        pan_center_steps="$(arg pan_center_steps)"
-        tilt_center_steps="$(arg tilt_center_steps)"
         sts3215_max_vel_steps="${sts3215_max_vel_steps}"
-        pan_joint_lower="${pan_joint_lower}"
-        pan_joint_upper="${pan_joint_upper}"
-        tilt_joint_lower="${tilt_joint_lower}"
-        tilt_joint_upper="${tilt_joint_upper}"
         ros2_control_hardware_type="$(arg ros2_control_hardware_type)"/>
   </ros2_control>

File: pt_description/urdf/pantilt.joints.xacro (robot description, xacro)
@@ -8,7 +8,7 @@
     block with the STSHardwareInterface plugin.
     Params:
-      pan_motor_id          — STS3215 motor ID for pan axis
+      shoulder_pan_motor_id — STS3215 motor ID for pan axis
       tilt_motor_id         — STS3215 motor ID for tilt axis
-      pan_center_steps      — raw step value (0–4095) for pan centre position
+      shoulder_pan_center_steps — raw step value (0–4095) for pan centre position
       tilt_center_steps     — raw step value (0–4095) for tilt centre position
       sts3215_max_vel_steps — motor's max velocity in steps/s, model-dependent;
@@ -16,11 +16,11 @@
   -->
   <xacro:macro name="pantilt_joints" params="
-      pan_motor_id:=1
+      shoulder_pan_motor_id:=1
       tilt_motor_id:=2
-      pan_center_steps:=2048
-      tilt_center_steps:=2646
+      shoulder_pan_center_steps:=2048
+      tilt_center_steps:=2048
       sts3215_max_vel_steps:=3400
-      pan_joint_lower:=-1.5708
-      pan_joint_upper:=1.5708
+      shoulder_pan_lower:=-1.5708
+      shoulder_pan_upper:=1.5708
       tilt_joint_lower:=-1.5708
       tilt_joint_upper:=1.5708
@@ -29,14 +29,14 @@
     <xacro:property name="pantilt_max_velocity_steps" value="${int(sts3215_max_vel_steps * 0.85)}"/>
     <xacro:property name="pantilt_max_velocity_rads"  value="${pantilt_max_velocity_steps * 2 * pi / 4096}"/>
-    <!-- Pan axis: rotates the payload around Z -->
-    <joint name="pan_joint">
-      <param name="motor_id">${pan_motor_id}</param>
+    <!-- Shoulder-pan axis: rotates the payload around Z -->
+    <joint name="shoulder_pan_joint">
+      <param name="motor_id">${shoulder_pan_motor_id}</param>
       <param name="operating_mode">0</param>
-      <param name="min_position">${pan_joint_lower}</param>
-      <param name="max_position">${pan_joint_upper}</param>
+      <param name="min_position">${shoulder_pan_lower}</param>
+      <param name="max_position">${shoulder_pan_upper}</param>
       <!-- Motor-specific, model-dependent parameter (per joint so different STS models can share this bus) -->
       <param name="max_velocity_steps">${sts3215_max_vel_steps}</param>
       <param name="max_velocity">${pantilt_max_velocity_rads}</param>
-      <param name="position_center_steps">${pan_center_steps}</param>
+      <param name="position_center_steps">${shoulder_pan_center_steps}</param>
       <command_interface name="position"/>
       <state_interface name="position"/>

File: pt_description/urdf/pantilt.module.xacro (robot description, xacro)
@@ -45,20 +45,20 @@
       </collision>
     </link>
-    <!-- Pan link -->
-    <link name="pan_link">
+    <!-- Shoulder link (was "pan_link") -->
+    <link name="shoulder_link">
       <inertial>
         <mass value="0.119226"/>
-        <origin xyz="-9.07886e-05 0.0590972 0.031089" rpy="0 0 0"/>
+        <origin xyz="-9.07886e-05 0.0590972 -0.0172669" rpy="0 0 0"/>
         <inertia ixx="5.94278e-05" ixy="0" ixz="0" iyy="5.89975e-05" iyz="0" izz="3.13712e-05"/>
       </inertial>
       <visual>
-        <origin xyz="${pan_joint_mesh_xyz}" rpy="${pan_joint_mesh_rpy}"/>
+        <origin xyz="${shoulder_pan_mesh_xyz}" rpy="${shoulder_pan_mesh_rpy}"/>
         <geometry>
-          <mesh filename="package://pt_description/meshes/${pan_joint_mesh}"/>
+          <mesh filename="package://pt_description/meshes/${shoulder_pan_mesh}"/>
         </geometry>
         <material name="light_grey"/>
       </visual>
       <visual>
-        <origin xyz="0 0 0" rpy="${pan_offset_rx} 0 ${pan_offset_rz}"/>
+        <origin xyz="0 0 -0.0483559" rpy="${shoulder_offset_rx} 0 ${shoulder_offset_rz}"/>
         <geometry>
           <mesh filename="package://pt_description/meshes/tilt_motor.stl"/>
@@ -67,7 +67,7 @@
       </visual>
       <collision>
-        <origin xyz="${pan_joint_mesh_xyz}" rpy="${pan_joint_mesh_rpy}"/>
+        <origin xyz="${shoulder_pan_mesh_xyz}" rpy="${shoulder_pan_mesh_rpy}"/>
         <geometry>
-          <mesh filename="package://pt_description/meshes/${pan_joint_mesh}"/>
+          <mesh filename="package://pt_description/meshes/${shoulder_pan_mesh}"/>
         </geometry>
       </collision>
@@ -98,15 +98,15 @@
          errors. gazebo mode: uses the real computed ceiling instead, since GazeboSimSystem
          actually enforces this limit on the simulated joint. -->
-    <!-- Pan joint (revolute) -->
-    <joint name="pan_joint" type="revolute">
+    <!-- Shoulder-pan joint (revolute; was "pan_joint") -->
+    <joint name="shoulder_pan_joint" type="revolute">
       <parent link="pantilt_base_link"/>
-      <child link="pan_link"/>
-      <origin xyz="${pan_joint_x} 0 ${pan_joint_z}" rpy="0 0 0"/>
+      <child link="shoulder_link"/>
+      <origin xyz="${shoulder_pan_x} 0 ${shoulder_pan_z}" rpy="0 0 0"/>
       <axis xyz="0 0 1"/>
-      <limit lower="${pan_joint_lower}" upper="${pan_joint_upper}" effort="${max_torque_nm}" velocity="${1e6 if '$(arg ros2_control_hardware_type)' == 'real' else pantilt_max_velocity_rads}"/>
+      <limit lower="${shoulder_pan_lower}" upper="${shoulder_pan_upper}" effort="${max_torque_nm}" velocity="${1e6 if '$(arg ros2_control_hardware_type)' == 'real' else pantilt_max_velocity_rads}"/>
     </joint>
     <!-- Tilt joint (revolute) -->
     <joint name="tilt_joint" type="revolute">
-      <parent link="pan_link"/>
+      <parent link="shoulder_link"/>
       <child link="tilt_link"/>
       <origin xyz="${tilt_joint_x} 0 ${tilt_joint_z}" rpy="${tilt_joint_rx} ${tilt_joint_ry} 0"/>

File: pt_description/urdf/pantilt.urdf.xacro (robot description, xacro)
@@ -5,8 +5,4 @@
   <xacro:arg name="use_mock"       default="false"/>
   <xacro:arg name="use_sync_write" default="true"/>
-  <xacro:arg name="pan_motor_id"   default="1"/>
-  <xacro:arg name="tilt_motor_id"  default="2"/>
-  <xacro:arg name="pan_center_steps" default="2048"/>
-  <xacro:arg name="tilt_center_steps" default="2646"/>
   <xacro:include filename="$(find pt_description)/urdf/pantilt.common.xacro"/>
   <xacro:include filename="$(find pt_description)/urdf/pantilt.control.xacro"/>

File: pt_description/urdf/pt100.urdf (robot description, URDF)
Before this commit: robot pantilt, 7 links, 6 joints
Links:
- removed link pan_link
- added link shoulder_link, mass 0.119226; collision mesh filename=../meshes/pan_joint_100.stl; visual mesh filename=../meshes/pan_joint_100.stl
Joints:
- removed joint pan_joint
- added joint shoulder_pan_joint: type revolute, parent pantilt_base_link, child shoulder_link, origin xyz=0.0452 0 0.0648559 rpy=0 0 0, axis 0 0 1, limit lower=-1.5708 upper=1.5708 effort=2.942 velocity=1000000.0
- joint tilt_joint: origin xyz=0.0306 0 0.1025 rpy=-1.5707963267948966 1.5707963267948966 0 -> xyz=0.0306 0 0.0541441 rpy=-1.5707963267948966 1.5707963267948966 0; parent pan_link -> shoulder_link
