Commit message: Align pt101/pt100 with so101/so100 conventions, add tests, single-source-of-truth config
Brings pantilt_ros2 closer to structural parity with so_arm_ros2 (treated as the
reference implementation for a repurposed SO-ARM100/101 first-two-joints device):

- Fix pan_joint's origin-to-mesh alignment: pan_link's own-link mesh bbox now sits
  relative to pan_joint's origin the same way SO101's shoulder_link sits relative to
  shoulder_pan_joint (verified via STL bounding-box measurement against so101.urdf).
  Zero world-space regression - pan_joint's axis was resliced with an equal-and-opposite
  compensation on pan_link's own mesh content, verified via mesh-vertex-world-position
  diff (max 2.8e-17m) and FK diff on tilt_joint/tilt_link/oak_link/oak_imu_frame (zero
  diff at rest and at arbitrary joint angles). pt100 needed no change - confirmed exact
  match (delta=0.0) to SO100's own convention already.

- Rename pan_joint/pan_link -> shoulder_pan_joint/shoulder_link (and matching internal
  xacro properties) to match so101/so100's own joint/link naming, across pt_description's
  URDF/xacro and MJCF files.

- Motor IDs, step-centering, and joint limits are no longer duplicated in
  pt_control/config/urdf_config.yaml - they're now baked into pantilt.joints.xacro's
  macro defaults as the single source of truth, matching so101.control.xacro/
  so100.control.xacro's convention. Also fixes a latent bug: the macro's own
  tilt_center_steps default was stale at 2646 (real value 2048), never visible since
  urdf_config.yaml always overrode it.

- controller-manager spawner naming: -c /controller_manager -> -c controller_manager,
  matching so_arm_control's relative naming.

- Add pt_description/test/test_urdf_xacro.py, modeled on so_arm_description's own -
  xacro-processing + XML-structure smoke tests (joint limits, ros2_control coverage,
  mesh existence, hardware-plugin selection, parent-child chain, MJCF processing).
  pt_description had no test suite before this.

- Add detect-private-key, check-added-large-files, and actionlint pre-commit hooks,
  matching so_arm_ros2's .pre-commit-config.yaml.

Regenerated pt101.urdf/pt100.urdf and the pt100/pt101_oakd_s2.xml MJCF snapshots to
match. lekiwi_ros2's own base_pantilt.* files and control.launch.py/urdf_config.yaml
updated to match in a companion commit there.

Co-Authored-By: Claude Sonnet 5 <noreply@anthropic.com>

File: pt_description/urdf/pt101.urdf (robot description, URDF)
Before this commit: robot pantilt, 7 links, 6 joints
Links:
- removed link pan_link
- added link shoulder_link, mass 0.119226; collision mesh filename=../meshes/pan_joint_101.stl; visual mesh filename=../meshes/pan_joint_101.stl
Joints:
- removed joint pan_joint
- added joint shoulder_pan_joint: type revolute, parent pantilt_base_link, child shoulder_link, origin xyz=0.0452 0 0.0648559 rpy=0 0 0, axis 0 0 1, limit lower=-1.5708 upper=1.5708 effort=2.942 velocity=1000000.0
- joint tilt_joint: origin xyz=0.0306 0 0.1025 rpy=-1.5707963267948966 1.5707963267948966 0 -> xyz=0.0306 0 0.0541441 rpy=-1.5707963267948966 1.5707963267948966 0; parent pan_link -> shoulder_link
